Commit message: Added better imu and meshes
Signed-off-by: Jakub Delicat <delicat.kuba@gmail.com>

File: quadruped_robot_description/urdf/gazebo.urdf.xacro (robot description, xacro)
@@ -5,4 +5,14 @@
       <parameters>$(find quadruped_controller)/config/jtc_controllers.yaml</parameters>
     </plugin>
+    <plugin filename="libignition-gazebo-detachable-joint-system.so" name="ignition::gazebo::systems::DetachableJoint">
+      <parent_link>rear_left_foot_link</parent_link>
+      <child_model>4BarBot</child_model>
+      <child_link>rear_left_chain_close_b_link</child_link>
+      <attach_topic>close_loop</attach_topic>
+    </plugin>
+    <!-- <plugin filename="libattach-links.so" name="ignition::gazebo::::systems::AttachLinks">
+      <parent>rear_left_chain_close_a_link</parent>
+      <child>rear_left_chain_close_b_link</child>
+    </plugin> -->
   </gazebo>
 </robot>

File: quadruped_robot_description/urdf/inertia.urdf.xacro (robot description, xacro)
@@ -22,6 +22,17 @@
     <inertial>
       <mass value="2e-06"/>
-      <inertia ixx="1.1e-14" ixy="0" ixz="0" iyy="1.1e-14" iyz="0" izz="1.1e-14"/>
+      <inertia ixx="1.1e-09" ixy="0" ixz="0" iyy="1.1e-09" iyz="0" izz="1.1e-09"/>
     </inertial>
   </xacro:macro>
+  <xacro:macro name="geometry_stub">
+        <origin rpy=" 0 0 0" xyz="0.0 0.0  0.0 " />
+        <geometry>
+          <box size="0.0001 0.0001 0.0001 "/>
+        </geometry>
+  </xacro:macro>
+  <xacro:macro name="grey_material">
+    <material name="grey">
+      <color rgba="0.5 0.5 0.5 1.0"/>
+    </material>
+  </xacro:macro>
 </robot>

File: quadruped_robot_description/urdf/leg.urdf.xacro (robot description, xacro)
@@ -31,5 +31,5 @@
       <origin xyz="0.031 0.0 0.0" rpy="${first_joint_offset} 0.0 0.0" />
       <axis xyz="1 0 0" />
-      <limit effort="2.0" lower="-3.1416" upper="3.1416" velocity="0.1" />
+      <limit effort="100.0" lower="-3.1416" upper="3.1416" velocity="10.0" />
       <dynamics damping="0.1" friction="0.1" />
     </joint>
@@ -38,5 +38,5 @@
     <xacro:property name="gear_ratio" value="0.166666" />
     <xacro:property name="second_joint_gear_correction" value="${0*gear_ratio*2*pi}" />
-    <xacro:property name="third_joint_gear_correction" value="${2*gear_ratio*2*pi}" />
+    <xacro:property name="third_joint_gear_correction" value="${3*gear_ratio*2*pi}" />
     <joint name="${prefix}_second_joint"
       type="revolute">
@@ -46,5 +46,5 @@
         rpy="0.0 0.0 ${pi + second_joint_gear_correction} " />
       <axis xyz="0 0 1" />
-      <limit effort="2.0" lower="1.57" upper="4.71" velocity="0.1" />
+      <limit effort="100.0" lower="1.57" upper="4.71" velocity="10.0" />
       <dynamics damping="0.1" friction="0.1" />
     </joint>
@@ -57,5 +57,5 @@
       <origin xyz="0.0 0.0 0.0555" rpy="0.0 0.0 ${third_joint_gear_correction_dir*third_joint_gear_correction}" />
       <axis xyz="0 0 1" />
-      <limit effort="2.0" lower="0.425" upper="5.8" velocity="0.1" />
+      <limit effort="100.0" lower="0.425" upper="5.8" velocity="10.0" />
       <dynamics damping="0.1" friction="0.1" />
     </joint>
@@ -68,5 +68,5 @@
       <origin xyz="0.125 0.0 0.0255" rpy="0.0 0.0 ${pi}" />
       <axis xyz="0 0 -1" />
-      <limit effort="  2.0" lower="-0.8" upper="-2.9" velocity="0.1" />
+      <limit effort="  2.0" lower="-0.8" upper="-2.9" velocity="10.0" />
       <dynamics damping="0.1" friction="0.1" />
     </joint>
@@ -79,8 +79,15 @@
       <origin xyz="-0.125 0.0 0.058" rpy="0.0 0.0 0.0" />
       <axis xyz="0 0 -1" />
-      <limit effort="5.0" lower="-3.14" upper="3.14" velocity="0.1" />
+      <limit effort="100.0" lower="-3.14" upper="3.14" velocity="10.0" />
       <dynamics damping="0.1" friction="0.1" />
     </joint>
     <link name="${prefix}_foot_link" >
+      <visual>
+        <xacro:geometry_stub/>
+        <xacro:grey_material />
+</visual>
+      <collision name="${prefix}_foot_link_collision">
+        <xacro:geometry_stub/>
+      </collision>
       <xacro:inertia_stub/>
     </link>
@@ -91,8 +98,15 @@
       <origin xyz="0.21 0.0 0.0115" rpy="0.0 0.0 0.0" />
       <axis xyz="0 0 1" />
-      <limit effort="2.0" lower="-3.14" upper="3.14" velocity="0.1" />
+      <limit effort="100.0" lower="-3.14" upper="3.14" velocity="10.0" />
       <dynamics damping="0.1" friction="0.1" />
     </joint>
     <link name="${prefix}_chain_close_a_link" >
+      <visual>
+        <xacro:geometry_stub/>
+        <xacro:grey_material />
+</visual>
+      <collision name="${prefix}_chain_close_a_link_collision">
+        <xacro:geometry_stub/>
+      </collision>
       <xacro:inertia_stub/>
     </link>
@@ -105,4 +119,11 @@
     </joint>
     <link name="${prefix}_chain_close_b_link">
+      <visual>
+        <xacro:geometry_stub/>
+        <xacro:grey_material />
+</visual>
+      <collision name="${prefix}_chain_close_b_link_collision">
+        <xacro:geometry_stub/>
+      </collision>
       <xacro:inertia_stub/>
     </link>
@@ -121,9 +142,10 @@
           <mesh filename="package://quadruped_robot_description/meshes/first_link.dae" />
         </geometry>
-      </visual>
-      <collision>
-        <origin rpy=" 0 ${pi/2} 0" xyz="0.01 0  0" />
-        <geometry>
-          <cylinder length="0.04" radius="0.05"/>
+        <xacro:grey_material />
+</visual>
+      <collision name="${name}_collision">
+        <origin rpy="0 0 0" xyz="0.0 0 0.0" />
+        <geometry>
+          <mesh filename="package://quadruped_robot_description/meshes/first_link.dae" />
         </geometry>
       </collision>
@@ -138,9 +160,10 @@
           <mesh filename="package://quadruped_robot_description/meshes/second_link.dae" />
         </geometry>
-      </visual>
-      <collision>
-        <origin rpy=" 0 0.0 0" xyz="0.055 0  0" />
-        <geometry>
-          <box size="0.11 0.1 0.065 "/>
+        <xacro:grey_material />
+</visual>
+      <collision name="${name}_collision">
+        <origin rpy="0 0 0" xyz="0.0 0 0.0" />
+        <geometry>
+          <mesh filename="package://quadruped_robot_description/meshes/second_link.dae" />
         </geometry>
       </collision>
@@ -155,9 +178,10 @@
           <mesh filename="package://quadruped_robot_description/meshes/third_link.dae" />
         </geometry>
-      </visual>
-      <collision>
-        <origin rpy=" 0 0 0" xyz="0.0 0 0.025  " />
-        <geometry>
-          <cylinder length="0.05" radius="0.05"/>
+        <xacro:grey_material />
+</visual>
+      <collision name="${name}_collision">
+       <origin rpy="0 0 0" xyz="0.0 0 0.0" />
+        <geometry>
+          <mesh filename="package://quadruped_robot_description/meshes/third_link.dae" />
         </geometry>
       </collision>
@@ -172,9 +196,10 @@
           <mesh filename="package://quadruped_robot_description/meshes/fourth_link.dae" />
         </geometry>
-      </visual>
-      <collision>
-        <origin rpy=" 0 0 0" xyz="0.0625 0.0  0.015 " />
-        <geometry>
-          <box size="0.175 0.04 0.025 "/>
+        <xacro:grey_material />
+</visual>
+      <collision name="${name}_collision">
+        <origin rpy="0 0 0" xyz="0.0 0 0.0" />
+        <geometry>
+          <mesh filename="package://quadruped_robot_description/meshes/fourth_link.dae" />
         </geometry>
       </collision>
@@ -189,9 +214,10 @@
           <mesh filename="package://quadruped_robot_description/meshes/fifth_link.dae" />
         </geometry>
-      </visual>
-      <collision>
-        <origin rpy=" 0 0 0" xyz="0.105 0.0  0.008 " />
-        <geometry>
-          <box size="0.25 0.04 0.0175 "/>
+        <xacro:grey_material />
+</visual>
+      <collision name="${name}_collision">
+         <origin rpy="0 0 0" xyz="0.0 0 0.0" />
+        <geometry>
+          <mesh filename="package://quadruped_robot_description/meshes/fifth_link.dae" />
         </geometry>
       </collision>
@@ -206,9 +232,10 @@
           <mesh filename="package://quadruped_robot_description/meshes/sixth_link.dae" />
         </geometry>
-      </visual>
-      <collision>
-        <origin rpy=" 0 0 0" xyz="0.105 0.0  0.008 " />
-        <geometry>
-          <box size="0.25 0.04 0.0175 "/>
+        <xacro:grey_material />
+</visual>
+      <collision name="${name}_collision">
+        <origin rpy="0 0 0" xyz="0.0 0 0.0" />
+        <geometry>
+          <mesh filename="package://quadruped_robot_description/meshes/sixth_link.dae" />
         </geometry>
       </collision>

File: quadruped_robot_description/urdf/quadruped_robot.urdf.xacro (robot description, xacro)
@@ -5,4 +5,7 @@
   <xacro:include filename="$(find quadruped_robot_description)/urdf/ros2_control.urdf.xacro" />
   <xacro:include filename="$(find quadruped_robot_description)/urdf/gazebo.urdf.xacro"  />
+  <mujoco>
+    <compiler meshdir="$(find quadruped_robot_description)/meshes" balanceinertia="true" discardvisual="false"/>
+  </mujoco>
   <xacro:arg name="use_hardware" default="True" />
   <xacro:arg name="use_sim" default="False" />
@@ -10,19 +13,19 @@
     <color rgba="0.5 0.5 0.5 1" />
   </material>
-  <!-- Define the base (body) -->
   <link name="base_link">
     <visual>
       <origin rpy="0 0 ${pi}" xyz="0.0 0 0" />
-      <geometry>
+      <geometry name="base_link">
         <mesh filename="package://quadruped_robot_description/meshes/base_link.dae" />
       </geometry>
+      <xacro:grey_material />
     </visual>
     <collision>
-      <origin xyz="0.01 0 0.06" />
-      <geometry>
-        <box size="0.59 0.225 0.10" />
+      <origin rpy="0 0 ${pi}" xyz="0.0 0 0" />
+      <geometry name="base_link">
+        <mesh filename="package://quadruped_robot_description/meshes/base_link.dae" />
       </geometry>
     </collision>
-    <xacro:box_inertia m="14.0" w="0.59" h="0.225" d="0.1" xyz="0.01 0 0.06" />
+    <xacro:box_inertia m="50.0" w="0.59" h="0.225" d="0.1" xyz="0.01 0 0.06" />
   </link>
   <link name="imu_link" />
@@ -32,5 +35,4 @@
     <origin xyz="0.0 0.0 0.1" rpy=" 0.0 ${pi} 0.0" />
   </joint>
-  <!-- Define the four legs -->
   <xacro:leg prefix="rear_left" xyz="-0.131 0.06 0.06" rpy="0 0 ${pi}" first_joint_offset="${pi}"
     third_joint_gear_correction_dir="-1.0" />
@@ -42,4 +44,5 @@
     third_joint_gear_correction_dir="1.0"
   />
-  <xacro:quadruperd_ros2_control use_hardware="$(arg use_hardware)" use_sim="$(arg use_sim)" />
+  <!-- <xacro:quadruperd_ros2_control use_hardware="$(arg use_hardware)" use_sim="$(arg use_sim)" /> -->
+  <xacro:imu_ros2_control/>
 </robot>

File: quadruped_robot_description/urdf/ros2_control.urdf.xacro (robot description, xacro)
@@ -41,4 +41,28 @@
         </joint>
     </xacro:macro>
+    <xacro:macro name="imu_ros2_control">
+        <ros2_control name="imu" type="sensor">
+            <hardware>
+                <plugin>bmx160_serial_hardware_interface/BMX160SerialHardwareInterface</plugin>
+                <param name="port">/dev/ttyACM0</param>
+                <param name="baud_rate">9600</param>
+            </hardware>
+            <sensor name="imu">
+                <state_interface name="orientation.x" />
+                <state_interface name="orientation.y" />
+                <state_interface name="orientation.z" />
+                <state_interface name="orientation.w" />
+                <state_interface name="magnetometer.x" />
+                <state_interface name="magnetometer.y" />
+                <state_interface name="magnetometer.z" />
+                <state_interface name="angular_velocity.x" />
+                <state_interface name="angular_velocity.y" />
+                <state_interface name="angular_velocity.z" />
+                <state_interface name="linear_acceleration.x" />
+                <state_interface name="linear_acceleration.y" />
+                <state_interface name="linear_acceleration.z" />
+            </sensor>
+        </ros2_control>
+    </xacro:macro>
     <xacro:macro name="quadruperd_ros2_control" params="use_hardware use_sim">
         <ros2_control name="MD80HardwareInterface" type="system">
@@ -80,11 +104,11 @@
                 ddq_kd="${kd2}" max_torque="${max_torque2}" />
             <xacro:ros2_control_joint_can name="front_right_third_joint" can_id="22" ddq_kp="${kp3}"
-                ddq_kd="${kd3}" max_torque="${max_torque3}"/>
+                ddq_kd="${kd3}" max_torque="${max_torque3}" />
             <xacro:ros2_control_joint_can name="rear_right_first_joint" can_id="30" ddq_kp="${kp1}"
                 ddq_kd="${kd1}" max_torque="15.0" />
             <xacro:ros2_control_joint_can name="rear_right_second_joint" can_id="31" ddq_kp="${kp2}"
-                ddq_kd="${kd2}" max_torque="${max_torque2}"/>
+                ddq_kd="${kd2}" max_torque="${max_torque2}" />
             <xacro:ros2_control_joint_can name="rear_right_third_joint" can_id="32" ddq_kp="${kp3}"
-                ddq_kd="${kd3}" max_torque="${max_torque3}"/>
+                ddq_kd="${kd3}" max_torque="${max_torque3}" />
             <!-- <xacro:ros2_control_passive_point name="rear_right_fourth_joint" />
     <xacro:ros2_control_passive_point name="rear_right_fifth_joint" /> -->
@@ -92,5 +116,5 @@
                 ddq_kd="${kd1}" max_torque="15.0" />
             <xacro:ros2_control_joint_can name="rear_left_second_joint" can_id="41" ddq_kp="${kp2}"
-                ddq_kd="${kd2}"  max_torque="${max_torque2}" />
+                ddq_kd="${kd2}" max_torque="${max_torque2}" />
             <xacro:ros2_control_joint_can name="rear_left_third_joint" can_id="42" ddq_kp="${kp3}"
                 ddq_kd="${kd3}" max_torque="${max_torque3}" />
