Commit message: Added docker and twist_to_traj
Signed-off-by: Jakub Delicat <delicat.kuba@gmail.com>

File: quadruped_robot_description/urdf/leg.urdf.xacro (robot description, xacro)
@@ -80,4 +80,20 @@
       <dynamics damping="0" friction="0" />
     </joint>
+    <link name="${prefix}_foot_first_link" />
+    <joint name="${prefix}_foot_first_joint"
+      type="fixed">
+      <parent link="${prefix}_sixth_link" />
+      <child link="${prefix}_foot_first_link" />
+      <origin xyz="0.21 0.0 0.0" rpy="0.0 0.0 0.0" />
+      <axis xyz="0 0 1" />
+    </joint>
+    <link name="${prefix}_foot_second_link" />
+    <joint name="${prefix}_foot_second_joint"
+      type="fixed">
+      <parent link="${prefix}_fifth_link" />
+      <child link="${prefix}_foot_second_link" />
+      <origin xyz="0.21 0.0 0.0" rpy="0.0 0.0 0.0" />
+      <axis xyz="0 0 1" />
+    </joint>
   </xacro:macro>
   <xacro:macro name="first_link" params="name">

File: quadruped_robot_description/urdf/quadruped_robot.urdf.xacro (robot description, xacro)
@@ -21,5 +21,5 @@
       <origin rpy="0 0 ${pi}" xyz="0.0 0 0.0" />
       <geometry>
-        <mesh filename="package://quadruped_robot_description/meshes/base_link.dae" />
+        <mesh filename="$package://quadruped_robot_description/meshes/base_link.dae" />
       </geometry>
     </collision>

File: quadruped_robot_description/urdf/ros2_control.urdf.xacro (robot description, xacro)
@@ -97,5 +97,5 @@
                 </xacro:if>
                 <xacro:unless value="${use_hardware}">
-                    <plugin>fake_components/GenericSystem</plugin>
+                    <plugin>mock_components/GenericSystem</plugin>
                 </xacro:unless>
                 <param name="port">/dev/ttyACM1</param>

Commit message: base XYZ kinematics | fixed Y leg kinematics
Signed-off-by: Jakub Delicat <delicat.kuba@gmail.com>

File: quadruped_robot_description/urdf/leg.urdf.xacro (robot description, xacro)
@@ -31,4 +31,5 @@
       <axis xyz="1 0 0" />
       <limit lower="-3.1416" upper="3.1416" effort="100" velocity="0.5" />
+      <dynamics damping="0.1" friction="0" />
     </joint>
     <xacro:third_link
@@ -45,5 +46,5 @@
       <axis xyz="0 0 1" />
       <limit lower="-3.14" upper="3.14" effort="100" velocity="0.5" />
-      <dynamics damping="0" friction="0" />
+      <dynamics damping="0.1" friction="0" />
     </joint>
     <xacro:fourth_link
@@ -56,5 +57,5 @@
       <axis xyz="0 0 1" />
       <limit lower="-3.14" upper="3.14" effort="100" velocity="0.5" />
-      <dynamics damping="0" friction="0" />
+      <dynamics damping="0.1" friction="0" />
     </joint>
     <xacro:fifth_link
@@ -112,7 +113,7 @@
       </collision>
       <inertial>
-        <mass value="0.5" />
-        <origin xyz="0 0 -0.2" />
-        <inertia ixx="0.05" ixy="0.0" ixz="0.0" iyy="0.05" iyz="0.0" izz="0.05" />
+        <mass value="0.05" />
+        <origin xyz="0 0 0" />
+        <inertia ixx="0.00005" ixy="0.0" ixz="0.0" iyy="0.00005" iyz="0.0" izz="0.00005" />
       </inertial>
     </link>
@@ -133,7 +134,7 @@
       </collision>
       <inertial>
-        <mass value="0.5" />
-        <origin xyz="0 0 -0.2" />
-        <inertia ixx="0.05" ixy="0.0" ixz="0.0" iyy="0.05" iyz="0.0" izz="0.05" />
+        <mass value="0.05" />
+        <origin xyz="0 0 0" />
+        <inertia ixx="0.00005" ixy="0.0" ixz="0.0" iyy="0.00005" iyz="0.0" izz="0.00005" />
       </inertial>
     </link>
@@ -154,7 +155,7 @@
       </collision>
       <inertial>
-        <mass value="0.5" />
-        <origin xyz="0 0 -0.2" />
-        <inertia ixx="0.05" ixy="0.0" ixz="0.0" iyy="0.05" iyz="0.0" izz="0.05" />
+        <mass value="0.05" />
+        <origin xyz="0 0 0" />
+        <inertia ixx="0.00005" ixy="0.0" ixz="0.0" iyy="0.00005" iyz="0.0" izz="0.00005" />
       </inertial>
     </link>
@@ -175,7 +176,7 @@
       </collision>
       <inertial>
-        <mass value="0.5" />
-        <origin xyz="0 0 -0.2" />
-        <inertia ixx="0.05" ixy="0.0" ixz="0.0" iyy="0.05" iyz="0.0" izz="0.05" />
+        <mass value="0.05" />
+        <origin xyz="0 0 0" />
+        <inertia ixx="0.00005" ixy="0.0" ixz="0.0" iyy="0.00005" iyz="0.0" izz="0.00005" />
       </inertial>
     </link>
@@ -196,7 +197,7 @@
       </collision>
       <inertial>
-        <mass value="0.5" />
-        <origin xyz="0 0 -0.2" />
-        <inertia ixx="0.05" ixy="0.0" ixz="0.0" iyy="0.05" iyz="0.0" izz="0.05" />
+        <mass value="0.05" />
+        <origin xyz="0 0 0" />
+        <inertia ixx="0.00005" ixy="0.0" ixz="0.0" iyy="0.00005" iyz="0.0" izz="0.00005" />
       </inertial>
     </link>
@@ -217,7 +218,7 @@
       </collision>
       <inertial>
-        <mass value="0.5" />
-        <origin xyz="0 0 -0.2" />
-        <inertia ixx="0.05" ixy="0.0" ixz="0.0" iyy="0.05" iyz="0.0" izz="0.05" />
+        <mass value="0.05" />
+        <origin xyz="0 0 0" />
+        <inertia ixx="0.00005" ixy="0.0" ixz="0.0" iyy="0.00005" iyz="0.0" izz="0.00005" />
       </inertial>
     </link>

File: quadruped_robot_description/urdf/quadruped_robot.urdf.xacro (robot description, xacro)
@@ -3,5 +3,7 @@
   <xacro:include filename="$(find quadruped_robot_description)/urdf/leg.urdf.xacro" />
   <xacro:include filename="$(find quadruped_robot_description)/urdf/ros2_control.urdf.xacro" />
+  <xacro:include filename="$(find quadruped_robot_description)/urdf/gazebo.urdf.xacro"  />
   <xacro:arg name="use_hardware" default="True" />
+  <xacro:arg name="use_sim" default="False" />
   <material name="grey">
     <color rgba="0.5 0.5 0.5 1" />
@@ -21,5 +23,5 @@
       <origin rpy="0 0 ${pi}" xyz="0.0 0 0.0" />
       <geometry>
-        <mesh filename="$package://quadruped_robot_description/meshes/base_link.dae" />
+        <mesh filename="package://quadruped_robot_description/meshes/base_link.dae" />
       </geometry>
     </collision>
@@ -46,4 +48,4 @@
     third_joint_gear_correction_dir="1.0"
   />
-  <xacro:quadruperd_ros2_control use_hardware="$(arg use_hardware)" />
+  <xacro:quadruperd_ros2_control use_hardware="$(arg use_hardware)" use_sim="$(arg use_sim)" />
 </robot>

File: quadruped_robot_description/urdf/ros2_control.urdf.xacro (robot description, xacro)
@@ -41,14 +41,19 @@
         </joint>
     </xacro:macro>
-    <xacro:macro name="quadruperd_ros2_control" params="use_hardware">
+    <xacro:macro name="quadruperd_ros2_control" params="use_hardware use_sim">
         <ros2_control name="MD80HardwareInterface" type="system">
             <hardware>
-                <xacro:if value="${use_hardware}">
-                    <plugin>md80_hardware_interface/MD80HardwareInterface</plugin>
-                    <param name="usb_port">/dev/ttyACM0</param>
-                    <param name="bus">spi</param>
+                <xacro:if value="${use_sim}">
+                    <plugin>ign_ros2_control/IgnitionSystem</plugin>
                 </xacro:if>
-                <xacro:unless value="${use_hardware}">
-                    <plugin>mock_components/GenericSystem</plugin>
+                <xacro:unless value="${use_sim}">
+                    <xacro:if value="${use_hardware}">
+                        <plugin>md80_hardware_interface/MD80HardwareInterface</plugin>
+                        <param name="usb_port">/dev/ttyACM0</param>
+                        <param name="bus">spi</param>
+                    </xacro:if>
+                    <xacro:unless value="${use_hardware}">
+                        <plugin>mock_components/GenericSystem</plugin>
+                    </xacro:unless>
                 </xacro:unless>
             </hardware>
@@ -93,45 +98,47 @@
     <xacro:ros2_control_passive_point name="rear_left_fifth_joint" /> -->
         </ros2_control>
-        <xacro:property name="mock_imu" value="sensor" />
-         <xacro:unless value="${use_hardware}">
-            <xacro:property name="mock_imu" value="system" />
+        <xacro:unless value="${use_sim}">
+            <xacro:property name="mock_imu" value="sensor" />
+            <xacro:unless value="${use_hardware}">
+                <xacro:property name="mock_imu" value="system" />
+            </xacro:unless>
+            <ros2_control name="imu" type="${mock_imu}">
+                <hardware>
+                    <xacro:if value="${use_hardware}">
+                        <plugin>bmx160_serial_hardware_interface/BMX160SerialHardwareInterface</plugin>
+                    </xacro:if>
+                    <xacro:unless value="${use_hardware}">
+                        <plugin>mock_components/GenericSystem</plugin>
+                    </xacro:unless>
+                    <param name="port">/dev/ttyACM0</param>
+                    <param name="baud_rate">9600</param>
+                    <!-- Madgwick Filter Params -->
+                    <!-- https://www.mouser.com/pdfdocs/BST-BMX160-DS000-11.pdf -->
+                    <!-- Output Noise 0.007 -->
+                    <!-- Bias stability 0.0000145 -->
+                    <param name="gain">0.003031089</param>
+                    <param name="zeta">0.000006279</param>
+                    <param name="mag_bias_x">0.002</param>
+                    <param name="mag_bias_y">0.002</param>
+                    <param name="mag_bias_z">0.002</param>
+                    <param name="world_frame">enu</param>
+                </hardware>
+                <sensor name="imu">
+                    <state_interface name="orientation.x" />
+                    <state_interface name="orientation.y" />
+                    <state_interface name="orientation.z" />
+                    <state_interface name="orientation.w" />
+                    <state_interface name="magnetometer.x" />
+                    <state_interface name="magnetometer.y" />
+                    <state_interface name="magnetometer.z" />
+                    <state_interface name="angular_velocity.x" />
+                    <state_interface name="angular_velocity.y" />
+                    <state_interface name="angular_velocity.z" />
+                    <state_interface name="linear_acceleration.x" />
+                    <state_interface name="linear_acceleration.y" />
+                    <state_interface name="linear_acceleration.z" />
+                </sensor>
+            </ros2_control>
         </xacro:unless>
-        <ros2_control name="imu" type="${mock_imu}">
-            <hardware>
-                <xacro:if value="${use_hardware}">
-                    <plugin>bmx160_serial_hardware_interface/BMX160SerialHardwareInterface</plugin>
-                </xacro:if>
-                <xacro:unless value="${use_hardware}">
-                    <plugin>mock_components/GenericSystem</plugin>
-                </xacro:unless>
-                <param name="port">/dev/ttyACM0</param>
-                <param name="baud_rate">9600</param>
-                <!-- Madgwick Filter Params -->
-                <!-- https://www.mouser.com/pdfdocs/BST-BMX160-DS000-11.pdf -->
-                <!-- Output Noise 0.007 -->
-                <!-- Bias stability 0.0000145 -->
-                <param name="gain">0.003031089</param>
-                <param name="zeta">0.000006279</param>
-                <param name="mag_bias_x">0.002</param>
-                <param name="mag_bias_y">0.002</param>
-                <param name="mag_bias_z">0.002</param>
-                <param name="world_frame">enu</param>
-            </hardware>
-            <sensor name="imu">
-                <state_interface name="orientation.x" />
-                <state_interface name="orientation.y" />
-                <state_interface name="orientation.z" />
-                <state_interface name="orientation.w" />
-                <state_interface name="magnetometer.x" />
-                <state_interface name="magnetometer.y" />
-                <state_interface name="magnetometer.z" />
-                <state_interface name="angular_velocity.x" />
-                <state_interface name="angular_velocity.y" />
-                <state_interface name="angular_velocity.z" />
-                <state_interface name="linear_acceleration.x" />
-                <state_interface name="linear_acceleration.y" />
-                <state_interface name="linear_acceleration.z" />
-            </sensor>
-        </ros2_control>
     </xacro:macro>
 </robot>

Commit message: better PD ks and joys from NUC
Signed-off-by: Jakub Delicat <delicat.kuba@gmail.com>

File: quadruped_robot_description/urdf/leg.urdf.xacro (robot description, xacro)
@@ -37,5 +37,5 @@
     <xacro:property name="gear_ratio" value="0.166666" />
     <xacro:property name="second_joint_gear_correction" value="${0*gear_ratio*2*pi}" />
-    <xacro:property name="third_joint_gear_correction" value="${3*gear_ratio*2*pi}" />
+    <xacro:property name="third_joint_gear_correction" value="${2*gear_ratio*2*pi}" />
     <joint name="${prefix}_second_joint"
       type="revolute">
@@ -86,5 +86,5 @@
       <parent link="${prefix}_sixth_link" />
       <child link="${prefix}_foot_first_link" />
-      <origin xyz="0.21 0.0 0.0" rpy="0.0 0.0 0.0" />
+      <origin xyz="0.21 0.0 0.0115" rpy="0.0 0.0 0.0" />
       <axis xyz="0 0 1" />
     </joint>
@@ -94,5 +94,5 @@
       <parent link="${prefix}_fifth_link" />
       <child link="${prefix}_foot_second_link" />
-      <origin xyz="0.21 0.0 0.0" rpy="0.0 0.0 0.0" />
+      <origin xyz="0.21 0.0 -0.0115" rpy="0.0 0.0 0.0" />
       <axis xyz="0 0 1" />
     </joint>

File: quadruped_robot_description/urdf/ros2_control.urdf.xacro (robot description, xacro)
@@ -51,5 +51,5 @@
                         <plugin>md80_hardware_interface/MD80HardwareInterface</plugin>
                         <param name="usb_port">/dev/ttyACM0</param>
-                        <param name="bus">spi</param>
+                        <param name="bus">usb</param>
                     </xacro:if>
                     <xacro:unless value="${use_hardware}">
@@ -58,13 +58,13 @@
                 </xacro:unless>
             </hardware>
-            <xacro:property name="kp1" value="80" />
-            <xacro:property name="kd1" value="12" />
+            <xacro:property name="kp1" value="25" />
+            <xacro:property name="kd1" value="5.0" />
             <!-- <xacro:property name="kp2" value="50" /> -->
-            <xacro:property name="kp2" value="50" />
-            <xacro:property name="kd2" value="10" />
+            <xacro:property name="kp2" value="7.5" />
+            <xacro:property name="kd2" value="1.0" />
             <xacro:property name="max_torque2" value="10.0" />
             <!-- <xacro:property name="kp3" value="50" /> -->
-            <xacro:property name="kp3" value="50" />
-            <xacro:property name="kd3" value="10" />
+            <xacro:property name="kp3" value="7.5" />
+            <xacro:property name="kd3" value="1.0" />
             <xacro:property name="max_torque3" value="10.0" />
             <xacro:ros2_control_joint_can name="front_left_first_joint" can_id="10" ddq_kp="${kp1}"
@@ -98,47 +98,4 @@
     <xacro:ros2_control_passive_point name="rear_left_fifth_joint" /> -->
         </ros2_control>
-        <xacro:unless value="${use_sim}">
-            <xacro:property name="mock_imu" value="sensor" />
-            <xacro:unless value="${use_hardware}">
-                <xacro:property name="mock_imu" value="system" />
-            </xacro:unless>
-            <ros2_control name="imu" type="${mock_imu}">
-                <hardware>
-                    <xacro:if value="${use_hardware}">
-                        <plugin>bmx160_serial_hardware_interface/BMX160SerialHardwareInterface</plugin>
-                    </xacro:if>
-                    <xacro:unless value="${use_hardware}">
-                        <plugin>mock_components/GenericSystem</plugin>
-                    </xacro:unless>
-                    <param name="port">/dev/ttyACM0</param>
-                    <param name="baud_rate">9600</param>
-                    <!-- Madgwick Filter Params -->
-                    <!-- https://www.mouser.com/pdfdocs/BST-BMX160-DS000-11.pdf -->
-                    <!-- Output Noise 0.007 -->
-                    <!-- Bias stability 0.0000145 -->
-                    <param name="gain">0.003031089</param>
-                    <param name="zeta">0.000006279</param>
-                    <param name="mag_bias_x">0.002</param>
-                    <param name="mag_bias_y">0.002</param>
-                    <param name="mag_bias_z">0.002</param>
-                    <param name="world_frame">enu</param>
-                </hardware>
-                <sensor name="imu">
-                    <state_interface name="orientation.x" />
-                    <state_interface name="orientation.y" />
-                    <state_interface name="orientation.z" />
-                    <state_interface name="orientation.w" />
-                    <state_interface name="magnetometer.x" />
-                    <state_interface name="magnetometer.y" />
-                    <state_interface name="magnetometer.z" />
-                    <state_interface name="angular_velocity.x" />
-                    <state_interface name="angular_velocity.y" />
-                    <state_interface name="angular_velocity.z" />
-                    <state_interface name="linear_acceleration.x" />
-                    <state_interface name="linear_acceleration.y" />
-                    <state_interface name="linear_acceleration.z" />
-                </sensor>
-            </ros2_control>
-        </xacro:unless>
     </xacro:macro>
 </robot>
