Commit message: Fixed collisions and inertias
Signed-off-by: Jakub Delicat <delicat.kuba@gmail.com>

File: quadruped_robot_description/urdf/leg.urdf.xacro (robot description, xacro)
@@ -1,4 +1,5 @@
 <?xml version="1.0"?>
 <robot xmlns:xacro="http://www.ros.org/wiki/xacro" name="quadruped_robot">
+  <xacro:include filename="$(find quadruped_robot_description)/urdf/inertia.urdf.xacro"  />
   <!-- Macro to define a leg -->
   <xacro:macro name="leg"
@@ -30,6 +31,6 @@
       <origin xyz="0.031 0.0 0.0" rpy="${first_joint_offset} 0.0 0.0" />
       <axis xyz="1 0 0" />
-      <limit lower="-3.1416" upper="3.1416" effort="100" velocity="0.5" />
-      <dynamics damping="0.1" friction="0" />
+      <limit effort="2.0" lower="-3.1416" upper="3.1416" velocity="0.1" />
+      <dynamics damping="0.1" friction="0.1" />
     </joint>
     <xacro:third_link
@@ -45,6 +46,6 @@
         rpy="0.0 0.0 ${pi + second_joint_gear_correction} " />
       <axis xyz="0 0 1" />
-      <limit lower="-3.14" upper="3.14" effort="100" velocity="0.5" />
-      <dynamics damping="0.1" friction="0" />
+      <limit effort="2.0" lower="1.57" upper="4.71" velocity="0.1" />
+      <dynamics damping="0.1" friction="0.1" />
     </joint>
     <xacro:fourth_link
@@ -56,43 +57,58 @@
       <origin xyz="0.0 0.0 0.0555" rpy="0.0 0.0 ${third_joint_gear_correction_dir*third_joint_gear_correction}" />
       <axis xyz="0 0 1" />
-      <limit lower="-3.14" upper="3.14" effort="100" velocity="0.5" />
-      <dynamics damping="0.1" friction="0" />
+      <limit effort="2.0" lower="0.425" upper="5.8" velocity="0.1" />
+      <dynamics damping="0.1" friction="0.1" />
     </joint>
     <xacro:fifth_link
       name="${prefix}_fifth_link" />
     <joint name="${prefix}_forth_joint"
-      type="continuous">
+      type="revolute">
       <parent link="${prefix}_fourth_link" />
       <child link="${prefix}_fifth_link" />
       <origin xyz="0.125 0.0 0.0255" rpy="0.0 0.0 ${pi}" />
       <axis xyz="0 0 -1" />
-      <limit lower="-3.14" upper="3.14" effort="100" velocity="0.5" />
-      <dynamics damping="0" friction="0" />
+      <limit effort="  2.0" lower="-0.8" upper="-2.9" velocity="0.1" />
+      <dynamics damping="0.1" friction="0.1" />
     </joint>
     <xacro:sixth_link
       name="${prefix}_sixth_link" />
     <joint name="${prefix}_fifth_joint"
-      type="continuous">
+      type="revolute">
       <parent link="${prefix}_third_link" />
       <child link="${prefix}_sixth_link" />
       <origin xyz="-0.125 0.0 0.058" rpy="0.0 0.0 0.0" />
       <axis xyz="0 0 -1" />
-      <limit lower="-3.14" upper="3.14" effort="100" velocity="0.5" />
-      <dynamics damping="0" friction="0" />
-    </joint>
-    <link name="${prefix}_foot_first_link" />
-    <joint name="${prefix}_foot_first_joint"
-      type="fixed">
+      <limit effort="5.0" lower="-3.14" upper="3.14" velocity="0.1" />
+      <dynamics damping="0.1" friction="0.1" />
+    </joint>
+    <link name="${prefix}_foot_link" >
+      <xacro:inertia_stub/>
+    </link>
+    <joint name="${prefix}_foot_joint"
+      type="revolute">
       <parent link="${prefix}_sixth_link" />
-      <child link="${prefix}_foot_first_link" />
+      <child link="${prefix}_foot_link" />
       <origin xyz="0.21 0.0 0.0115" rpy="0.0 0.0 0.0" />
       <axis xyz="0 0 1" />
-    </joint>
-    <link name="${prefix}_foot_second_link" />
-    <joint name="${prefix}_foot_second_joint"
+      <limit effort="2.0" lower="-3.14" upper="3.14" velocity="0.1" />
+      <dynamics damping="0.1" friction="0.1" />
+    </joint>
+    <link name="${prefix}_chain_close_a_link" >
+      <xacro:inertia_stub/>
+    </link>
+    <joint name="${prefix}_chain_close_a_joint"
       type="fixed">
       <parent link="${prefix}_fifth_link" />
-      <child link="${prefix}_foot_second_link" />
-      <origin xyz="0.21 0.0 -0.0115" rpy="0.0 0.0 0.0" />
+      <child link="${prefix}_chain_close_a_link" />
+      <origin xyz="0.105 0.0 -0.0115" rpy="0.0 0.0 0.0" />
+      <axis xyz="0 0 1" />
+    </joint>
+    <link name="${prefix}_chain_close_b_link">
+      <xacro:inertia_stub/>
+    </link>
+    <joint name="${prefix}_chain_close_b_joint" type="fixed">
+      <parent link="${prefix}_foot_link" />
+      <child link="${prefix}_chain_close_b_link" />
+      <origin rpy="0.0 0.0 0.0" xyz="0.105 0.0 0.0" />
       <axis xyz="0 0 1" />
     </joint>
@@ -107,14 +123,10 @@
       </visual>
       <collision>
-        <origin rpy="0 0 0" xyz="0.0 0 0.0" />
-        <geometry>
-          <mesh filename="package://quadruped_robot_description/meshes/first_link.dae" />
-        </geometry>
-      </collision>
-      <inertial>
-        <mass value="0.05" />
-        <origin xyz="0 0 0" />
-        <inertia ixx="0.00005" ixy="0.0" ixz="0.0" iyy="0.00005" iyz="0.0" izz="0.00005" />
-      </inertial>
+        <origin rpy=" 0 ${pi/2} 0" xyz="0.01 0  0" />
+        <geometry>
+          <cylinder length="0.04" radius="0.05"/>
+        </geometry>
+      </collision>
+      <xacro:cylinder_inertia m="0.6" r="0.05" h="0.04" />
     </link>
   </xacro:macro>
@@ -128,14 +140,10 @@
       </visual>
       <collision>
-        <origin rpy="0 0 0" xyz="0.0 0 0.0" />
-        <geometry>
-          <mesh filename="package://quadruped_robot_description/meshes/second_link.dae" />
-        </geometry>
-      </collision>
-      <inertial>
-        <mass value="0.05" />
-        <origin xyz="0 0 0" />
-        <inertia ixx="0.00005" ixy="0.0" ixz="0.0" iyy="0.00005" iyz="0.0" izz="0.00005" />
-      </inertial>
+        <origin rpy=" 0 0.0 0" xyz="0.055 0  0" />
+        <geometry>
+          <box size="0.11 0.1 0.065 "/>
+        </geometry>
+      </collision>
+      <xacro:cylinder_inertia m="0.6" r="0.05" h="0.04" xyz="0.055 0  0" />
     </link>
   </xacro:macro>
@@ -149,14 +157,10 @@
       </visual>
       <collision>
-        <origin rpy="0 0 0" xyz="0.0 0 0.0" />
-        <geometry>
-          <mesh filename="package://quadruped_robot_description/meshes/third_link.dae" />
-        </geometry>
-      </collision>
-      <inertial>
-        <mass value="0.05" />
-        <origin xyz="0 0 0" />
-        <inertia ixx="0.00005" ixy="0.0" ixz="0.0" iyy="0.00005" iyz="0.0" izz="0.00005" />
-      </inertial>
+        <origin rpy=" 0 0 0" xyz="0.0 0 0.025  " />
+        <geometry>
+          <cylinder length="0.05" radius="0.05"/>
+        </geometry>
+      </collision>
+      <xacro:cylinder_inertia m="0.6" r="0.05" h="0.04" xyz="0.0 0  0.025" />
     </link>
   </xacro:macro>
@@ -170,14 +174,10 @@
       </visual>
       <collision>
-        <origin rpy="0 0 0" xyz="0.0 0 0.0" />
-        <geometry>
-          <mesh filename="package://quadruped_robot_description/meshes/third_link.dae" />
-        </geometry>
-      </collision>
-      <inertial>
-        <mass value="0.05" />
-        <origin xyz="0 0 0" />
-        <inertia ixx="0.00005" ixy="0.0" ixz="0.0" iyy="0.00005" iyz="0.0" izz="0.00005" />
-      </inertial>
+        <origin rpy=" 0 0 0" xyz="0.0625 0.0  0.015 " />
+        <geometry>
+          <box size="0.175 0.04 0.025 "/>
+        </geometry>
+      </collision>
+      <xacro:box_inertia m="0.04" w="0.175" h="0.025" d="0.0175" xyz="0.0625 0.0  0.015" />
     </link>
   </xacro:macro>
@@ -191,14 +191,10 @@
       </visual>
       <collision>
-        <origin rpy="0 0 0" xyz="0.0 0 0.0" />
-        <geometry>
-          <mesh filename="package://quadruped_robot_description/meshes/fifth_link.dae" />
-        </geometry>
-      </collision>
-      <inertial>
-        <mass value="0.05" />
-        <origin xyz="0 0 0" />
-        <inertia ixx="0.00005" ixy="0.0" ixz="0.0" iyy="0.00005" iyz="0.0" izz="0.00005" />
-      </inertial>
+        <origin rpy=" 0 0 0" xyz="0.105 0.0  0.008 " />
+        <geometry>
+          <box size="0.25 0.04 0.0175 "/>
+        </geometry>
+      </collision>
+      <xacro:box_inertia m="0.05" w="0.25" h="0.04" d="0.0175" xyz="0.105 0  0.0" />
     </link>
   </xacro:macro>
@@ -212,14 +208,10 @@
       </visual>
       <collision>
-        <origin rpy="0 0 0" xyz="0.0 0 0.0" />
-        <geometry>
-          <mesh filename="package://quadruped_robot_description/meshes/sixth_link.dae" />
-        </geometry>
-      </collision>
-      <inertial>
-        <mass value="0.05" />
-        <origin xyz="0 0 0" />
-        <inertia ixx="0.00005" ixy="0.0" ixz="0.0" iyy="0.00005" iyz="0.0" izz="0.00005" />
-      </inertial>
+        <origin rpy=" 0 0 0" xyz="0.105 0.0  0.008 " />
+        <geometry>
+          <box size="0.25 0.04 0.0175 "/>
+        </geometry>
+      </collision>
+      <xacro:box_inertia m="0.05" w="0.25" h="0.04" d="0.0175" xyz="0.105 0  0.0" />
     </link>
   </xacro:macro>

File: quadruped_robot_description/urdf/quadruped_robot.urdf.xacro (robot description, xacro)
@@ -1,4 +1,5 @@
 <?xml version="1.0"?>
 <robot name="quadruped" xmlns:xacro="http://www.ros.org/wiki/xacro">
+  <xacro:include filename="$(find quadruped_robot_description)/urdf/inertia.urdf.xacro"  />
   <xacro:include filename="$(find quadruped_robot_description)/urdf/leg.urdf.xacro" />
   <xacro:include filename="$(find quadruped_robot_description)/urdf/ros2_control.urdf.xacro" />
@@ -16,19 +17,12 @@
         <mesh filename="package://quadruped_robot_description/meshes/base_link.dae" />
       </geometry>
-      <!-- <geometry>
-        <box size="0.25 0.23 0.06" />
-      </geometry> -->
     </visual>
     <collision>
-      <origin rpy="0 0 ${pi}" xyz="0.0 0 0.0" />
+      <origin xyz="0.01 0 0.06" />
       <geometry>
-        <mesh filename="package://quadruped_robot_description/meshes/base_link.dae" />
+        <box size="0.59 0.225 0.10" />
       </geometry>
     </collision>
-    <inertial>
-      <mass value="14.0" />
-      <origin xyz="0 0 0" />
-      <inertia ixx="0.1" ixy="0.0" ixz="0.0" iyy="0.1" iyz="0.0" izz="0.1" />
-    </inertial>
+    <xacro:box_inertia m="14.0" w="0.59" h="0.225" d="0.1" xyz="0.01 0 0.06" />
   </link>
   <link name="imu_link" />

Commit message: before defence
Signed-off-by: Jakub Delicat <delicat.kuba@gmail.com>

File: quadruped_robot_description/urdf/leg.urdf.xacro (robot description, xacro)
@@ -36,5 +36,5 @@
     <xacro:third_link
       name="${prefix}_third_link" />
-    <xacro:property name="gear_ratio" value="0.166666" />
+    <xacro:property name="gear_ratio" value="0.0" />
     <xacro:property name="second_joint_gear_correction" value="${0*gear_ratio*2*pi}" />
     <xacro:property name="third_joint_gear_correction" value="${3*gear_ratio*2*pi}" />
@@ -233,5 +233,5 @@
         </geometry>
         <xacro:grey_material />
-</visual>
+      </visual>
       <collision name="${name}_collision">
         <origin rpy="0 0 0" xyz="0.0 0 0.0" />

File: quadruped_robot_description/urdf/ros2_control.urdf.xacro (robot description, xacro)
@@ -7,5 +7,5 @@
               ddq_kp=1.0  ddq_kd=0.15">
         <joint name="${name}">
-            <command_interface name="position" />
+            <command_interface name="effort" />
             <state_interface name="position">
                 <param name="initial_value">0.0</param>
@@ -93,4 +93,5 @@
             <xacro:property name="kd3" value="1.0" />
             <xacro:property name="max_torque3" value="10.0" />
+<!--
             <xacro:ros2_control_joint_can name="front_left_first_joint" can_id="10" ddq_kp="${kp1}"
                 ddq_kd="${kd1}" max_torque="${max_torque1}" />
@@ -111,13 +112,13 @@
                 ddq_kd="${kd2}" max_torque="${max_torque2}" />
             <xacro:ros2_control_joint_can name="rear_right_third_joint" can_id="32" ddq_kp="${kp3}"
-                ddq_kd="${kd3}" max_torque="${max_torque3}" />
+                ddq_kd="${kd3}" max_torque="${max_torque3}" /> -->
             <!-- <xacro:ros2_control_passive_point name="rear_right_fourth_joint" />
     <xacro:ros2_control_passive_point name="rear_right_fifth_joint" /> -->
             <xacro:ros2_control_joint_can name="rear_left_first_joint" can_id="40" ddq_kp="${kp1}"
                 ddq_kd="${kd1}" max_torque="${max_torque1}" />
-            <xacro:ros2_control_joint_can name="rear_left_second_joint" can_id="41" ddq_kp="${kp2}"
+            <!-- <xacro:ros2_control_joint_can name="rear_left_second_joint" can_id="41" ddq_kp="${kp2}"
                 ddq_kd="${kd2}" max_torque="${max_torque2}" />
             <xacro:ros2_control_joint_can name="rear_left_third_joint" can_id="42" ddq_kp="${kp3}"
-                ddq_kd="${kd3}" max_torque="${max_torque3}" />
+                ddq_kd="${kd3}" max_torque="${max_torque3}" /> -->
             <!-- <xacro:ros2_control_passive_point name="rear_left_fourth_joint" />
     <xacro:ros2_control_passive_point name="rear_left_fifth_joint" /> -->

Commit message: Set  0 position
Signed-off-by: Jakub Delicat <delicat.kuba@gmail.com>

File: quadruped_robot_description/urdf/leg.urdf.xacro (robot description, xacro)
@@ -1,5 +1,5 @@
 <?xml version="1.0"?>
 <robot xmlns:xacro="http://www.ros.org/wiki/xacro" name="quadruped_robot">
-  <xacro:include filename="$(find quadruped_robot_description)/urdf/inertia.urdf.xacro"  />
+  <xacro:include filename="$(find quadruped_robot_description)/urdf/inertia.urdf.xacro" />
   <!-- Macro to define a leg -->
   <xacro:macro name="leg"
@@ -37,6 +37,6 @@
       name="${prefix}_third_link" />
     <xacro:property name="gear_ratio" value="0.0" />
-    <xacro:property name="second_joint_gear_correction" value="${0*gear_ratio*2*pi}" />
-    <xacro:property name="third_joint_gear_correction" value="${3*gear_ratio*2*pi}" />
+    <xacro:property name="second_joint_gear_correction" value="${third_joint_gear_correction_dir*0.3559}" />
+    <xacro:property name="third_joint_gear_correction" value="${-0.8+pi}" />
     <joint name="${prefix}_second_joint"
       type="revolute">
@@ -55,5 +55,6 @@
       <parent link="${prefix}_third_link" />
       <child link="${prefix}_fourth_link" />
-      <origin xyz="0.0 0.0 0.0555" rpy="0.0 0.0 ${third_joint_gear_correction_dir*third_joint_gear_correction}" />
+      <origin xyz="0.0 0.0 0.0555"
+        rpy="0.0 0.0 ${third_joint_gear_correction_dir*third_joint_gear_correction}" />
       <axis xyz="0 0 1" />
       <limit effort="100.0" lower="0.425" upper="5.8" velocity="10.0" />
@@ -62,5 +63,5 @@
     <xacro:fifth_link
       name="${prefix}_fifth_link" />
-    <joint name="${prefix}_forth_joint"
+    <joint name="${prefix}_fourth_joint"
       type="revolute">
       <parent link="${prefix}_fourth_link" />
@@ -82,56 +83,4 @@
       <dynamics damping="0.1" friction="0.1" />
     </joint>
-    <link name="${prefix}_foot_link" >
-      <visual>
-        <xacro:geometry_stub/>
-        <xacro:grey_material />
-</visual>
-      <collision name="${prefix}_foot_link_collision">
-        <xacro:geometry_stub/>
-      </collision>
-      <xacro:inertia_stub/>
-    </link>
-    <joint name="${prefix}_foot_joint"
-      type="revolute">
-      <parent link="${prefix}_sixth_link" />
-      <child link="${prefix}_foot_link" />
-      <origin xyz="0.21 0.0 0.0115" rpy="0.0 0.0 0.0" />
-      <axis xyz="0 0 1" />
-      <limit effort="100.0" lower="-3.14" upper="3.14" velocity="10.0" />
-      <dynamics damping="0.1" friction="0.1" />
-    </joint>
-    <link name="${prefix}_chain_close_a_link" >
-      <visual>
-        <xacro:geometry_stub/>
-        <xacro:grey_material />
-</visual>
-      <collision name="${prefix}_chain_close_a_link_collision">
-        <xacro:geometry_stub/>
-      </collision>
-      <xacro:inertia_stub/>
-    </link>
-    <joint name="${prefix}_chain_close_a_joint"
-      type="fixed">
-      <parent link="${prefix}_fifth_link" />
-      <child link="${prefix}_chain_close_a_link" />
-      <origin xyz="0.105 0.0 -0.0115" rpy="0.0 0.0 0.0" />
-      <axis xyz="0 0 1" />
-    </joint>
-    <link name="${prefix}_chain_close_b_link">
-      <visual>
-        <xacro:geometry_stub/>
-        <xacro:grey_material />
-</visual>
-      <collision name="${prefix}_chain_close_b_link_collision">
-        <xacro:geometry_stub/>
-      </collision>
-      <xacro:inertia_stub/>
-    </link>
-    <joint name="${prefix}_chain_close_b_joint" type="fixed">
-      <parent link="${prefix}_foot_link" />
-      <child link="${prefix}_chain_close_b_link" />
-      <origin rpy="0.0 0.0 0.0" xyz="0.105 0.0 0.0" />
-      <axis xyz="0 0 1" />
-    </joint>
   </xacro:macro>
   <xacro:macro name="first_link" params="name">
@@ -143,5 +92,5 @@
         </geometry>
         <xacro:grey_material />
-</visual>
+      </visual>
       <collision name="${name}_collision">
         <origin rpy="0 0 0" xyz="0.0 0 0.0" />
@@ -161,5 +110,5 @@
         </geometry>
         <xacro:grey_material />
-</visual>
+      </visual>
       <collision name="${name}_collision">
         <origin rpy="0 0 0" xyz="0.0 0 0.0" />
@@ -179,7 +128,7 @@
         </geometry>
         <xacro:grey_material />
-</visual>
+      </visual>
       <collision name="${name}_collision">
-       <origin rpy="0 0 0" xyz="0.0 0 0.0" />
+        <origin rpy="0 0 0" xyz="0.0 0 0.0" />
         <geometry>
           <mesh filename="package://quadruped_robot_description/meshes/third_link.dae" />
@@ -197,5 +146,5 @@
         </geometry>
         <xacro:grey_material />
-</visual>
+      </visual>
       <collision name="${name}_collision">
         <origin rpy="0 0 0" xyz="0.0 0 0.0" />
@@ -215,7 +164,7 @@
         </geometry>
         <xacro:grey_material />
-</visual>
+      </visual>
       <collision name="${name}_collision">
-         <origin rpy="0 0 0" xyz="0.0 0 0.0" />
+        <origin rpy="0 0 0" xyz="0.0 0 0.0" />
         <geometry>
           <mesh filename="package://quadruped_robot_description/meshes/fifth_link.dae" />

File: quadruped_robot_description/urdf/ros2_control.urdf.xacro (robot description, xacro)
@@ -93,5 +93,4 @@
             <xacro:property name="kd3" value="1.0" />
             <xacro:property name="max_torque3" value="10.0" />
-<!--
             <xacro:ros2_control_joint_can name="front_left_first_joint" can_id="10" ddq_kp="${kp1}"
                 ddq_kd="${kd1}" max_torque="${max_torque1}" />
@@ -112,15 +111,11 @@
                 ddq_kd="${kd2}" max_torque="${max_torque2}" />
             <xacro:ros2_control_joint_can name="rear_right_third_joint" can_id="32" ddq_kp="${kp3}"
-                ddq_kd="${kd3}" max_torque="${max_torque3}" /> -->
-            <!-- <xacro:ros2_control_passive_point name="rear_right_fourth_joint" />
-    <xacro:ros2_control_passive_point name="rear_right_fifth_joint" /> -->
+                ddq_kd="${kd3}" max_torque="${max_torque3}" />
             <xacro:ros2_control_joint_can name="rear_left_first_joint" can_id="40" ddq_kp="${kp1}"
                 ddq_kd="${kd1}" max_torque="${max_torque1}" />
-            <!-- <xacro:ros2_control_joint_can name="rear_left_second_joint" can_id="41" ddq_kp="${kp2}"
+            <xacro:ros2_control_joint_can name="rear_left_second_joint" can_id="41" ddq_kp="${kp2}"
                 ddq_kd="${kd2}" max_torque="${max_torque2}" />
             <xacro:ros2_control_joint_can name="rear_left_third_joint" can_id="42" ddq_kp="${kp3}"
-                ddq_kd="${kd3}" max_torque="${max_torque3}" /> -->
-            <!-- <xacro:ros2_control_passive_point name="rear_left_fourth_joint" />
-    <xacro:ros2_control_passive_point name="rear_left_fifth_joint" /> -->
+                ddq_kd="${kd3}" max_torque="${max_torque3}" />
         </ros2_control>
     </xacro:macro>

Commit message: Before removing inv
Signed-off-by: Jakub Delicat <delicat.kuba@gmail.com>

File: quadruped_robot_description/urdf/leg.urdf.xacro (robot description, xacro)
@@ -37,6 +37,6 @@
       name="${prefix}_third_link" />
     <xacro:property name="gear_ratio" value="0.0" />
-    <xacro:property name="second_joint_gear_correction" value="${third_joint_gear_correction_dir*0.3559}" />
-    <xacro:property name="third_joint_gear_correction" value="${-0.8+pi}" />
+    <xacro:property name="second_joint_gear_correction" value="${third_joint_gear_correction_dir*0.2793}" />
+    <xacro:property name="third_joint_gear_correction" value="${-1.117+pi}" />
     <joint name="${prefix}_second_joint"
       type="revolute">

File: quadruped_robot_description/urdf/ros2_control.urdf.xacro (robot description, xacro)
@@ -84,14 +84,14 @@
             <xacro:property name="kp1" value="25" />
             <xacro:property name="kd1" value="5.0" />
-            <xacro:property name="max_torque1" value="15.0" />
+            <xacro:property name="max_torque1" value="1.0" />
             <!-- <xacro:property name="kp2" value="50" /> -->
             <xacro:property name="kp2" value="7.5" />
             <xacro:property name="kd2" value="1.0" />
-            <xacro:property name="max_torque2" value="10.0" />
+            <xacro:property name="max_torque2" value="1.0" />
             <!-- <xacro:property name="kp3" value="50" /> -->
             <xacro:property name="kp3" value="7.5" />
             <xacro:property name="kd3" value="1.0" />
-            <xacro:property name="max_torque3" value="10.0" />
-            <xacro:ros2_control_joint_can name="front_left_first_joint" can_id="10" ddq_kp="${kp1}"
+            <xacro:property name="max_torque3" value="1.0" />
+            <!-- <xacro:ros2_control_joint_can name="front_left_first_joint" can_id="10" ddq_kp="${kp1}"
                 ddq_kd="${kd1}" max_torque="${max_torque1}" />
             <xacro:ros2_control_joint_can name="front_left_second_joint" can_id="11" ddq_kp="${kp2}"
@@ -111,5 +111,5 @@
                 ddq_kd="${kd2}" max_torque="${max_torque2}" />
             <xacro:ros2_control_joint_can name="rear_right_third_joint" can_id="32" ddq_kp="${kp3}"
-                ddq_kd="${kd3}" max_torque="${max_torque3}" />
+                ddq_kd="${kd3}" max_torque="${max_torque3}" /> -->
             <xacro:ros2_control_joint_can name="rear_left_first_joint" can_id="40" ddq_kp="${kp1}"
                 ddq_kd="${kd1}" max_torque="${max_torque1}" />
