Commit message: Fixed kinematics | still error with inverse
Signed-off-by: Jakub Delicat <delicat.kuba@gmail.com>

File: quadruped_robot_description/urdf/leg.urdf.xacro (robot description, xacro)
@@ -37,4 +37,6 @@
       name="${prefix}_third_link" />
     <xacro:property name="gear_ratio" value="0.0" />
+    <!-- <xacro:property name="second_joint_gear_correction" value="${third_joint_gear_correction_dir*0.2793}" />
+    <xacro:property name="third_joint_gear_correction" value="${-1.117+pi}" /> -->
     <xacro:property name="second_joint_gear_correction" value="${third_joint_gear_correction_dir*0.2793}" />
     <xacro:property name="third_joint_gear_correction" value="${-1.117+pi}" />

File: quadruped_robot_description/urdf/ros2_control.urdf.xacro (robot description, xacro)
@@ -7,5 +7,5 @@
               ddq_kp=1.0  ddq_kd=0.15">
         <joint name="${name}">
-            <command_interface name="effort" />
+            <command_interface name="acceleration" />
             <state_interface name="position">
                 <param name="initial_value">0.0</param>
@@ -29,14 +29,4 @@
             <param name="ddq_kp">${ddq_kp}</param>
             <param name="ddq_kd">${ddq_kd}</param>
-        </joint>
-    </xacro:macro>
-    <xacro:macro name="ros2_control_passive_point" params="name">
-        <joint name="${name}">
-            <state_interface name="position" />
-            <!-- TODO @delipl
-       <state_interface name="velocity">
-        <param name="initial_value">0.0</param>
-      </state_interface> -->
-            <!-- <state_interface name="effort" /> -->
         </joint>
     </xacro:macro>
@@ -79,4 +69,5 @@
                     <xacro:unless value="${use_hardware}">
                         <plugin>mock_components/GenericSystem</plugin>
+                        <param name="calculate_dynamics">true</param>
                     </xacro:unless>
                 </xacro:unless>
