Commit message: Added quadbar_kinematics
Signed-off-by: Jakub Delicat <delicat.kuba@gmail.com>

File: quadruped_robot_description/urdf/ros2_control.urdf.xacro (robot description, xacro)
@@ -44,5 +44,4 @@
         <ros2_control name="MD80HardwareInterface" type="system">
             <hardware>
-                <!-- <plugin>md80_hardware_interface/MD80HardwareInterface</plugin> -->
                 <xacro:if value="${use_hardware}">
                     <plugin>md80_hardware_interface/MD80HardwareInterface</plugin>
@@ -88,7 +87,16 @@
     <xacro:ros2_control_passive_point name="rear_left_fifth_joint" /> -->
         </ros2_control>
-        <ros2_control name="imu" type="sensor">
+        <xacro:property name="mock_imu" value="sensor" />
+         <xacro:unless value="${use_hardware}">
+            <xacro:property name="mock_imu" value="system" />
+        </xacro:unless>
+        <ros2_control name="imu" type="${mock_imu}">
             <hardware>
-                <plugin>bmx160_serial_hardware_interface/BMX160SerialHardwareInterface</plugin>
+                <xacro:if value="${use_hardware}">
+                    <plugin>bmx160_serial_hardware_interface/BMX160SerialHardwareInterface</plugin>
+                </xacro:if>
+                <xacro:unless value="${use_hardware}">
+                    <plugin>fake_components/GenericSystem</plugin>
+                </xacro:unless>
                 <param name="port">/dev/ttyACM1</param>
                 <param name="baud_rate">9600</param>

Commit message: Changes
Signed-off-by: Jakub Delicat <delicat.kuba@gmail.com>

File: quadruped_robot_description/urdf/ros2_control.urdf.xacro (robot description, xacro)
@@ -46,4 +46,5 @@
                 <xacro:if value="${use_hardware}">
                     <plugin>md80_hardware_interface/MD80HardwareInterface</plugin>
+                    <param name="usb_port">/dev/ttyACM0</param>
                 </xacro:if>
                 <xacro:unless value="${use_hardware}">
@@ -53,7 +54,9 @@
             <xacro:property name="kp1" value="80" />
             <xacro:property name="kd1" value="12" />
+            <!-- <xacro:property name="kp2" value="50" /> -->
             <xacro:property name="kp2" value="50" />
             <xacro:property name="kd2" value="10" />
-            <xacro:property name="kp3" value="50" />
+            <!-- <xacro:property name="kp3" value="50" /> -->
+            <xacro:property name="kp3" value="25" />
             <xacro:property name="kd3" value="10" />
             <xacro:ros2_control_joint_can name="front_left_first_joint" can_id="10" ddq_kp="${kp1}"

Commit message: Fixed forward kinematics
Signed-off-by: Jakub Delicat <delicat.kuba@gmail.com>

File: quadruped_robot_description/urdf/ros2_control.urdf.xacro (robot description, xacro)
@@ -84,13 +84,13 @@
             <xacro:property name="kp1" value="25" />
             <xacro:property name="kd1" value="5.0" />
-            <xacro:property name="max_torque1" value="1.0" />
+            <xacro:property name="max_torque1" value="3.0" />
             <!-- <xacro:property name="kp2" value="50" /> -->
             <xacro:property name="kp2" value="7.5" />
             <xacro:property name="kd2" value="1.0" />
-            <xacro:property name="max_torque2" value="1.0" />
+            <xacro:property name="max_torque2" value="3.0" />
             <!-- <xacro:property name="kp3" value="50" /> -->
             <xacro:property name="kp3" value="7.5" />
             <xacro:property name="kd3" value="1.0" />
-            <xacro:property name="max_torque3" value="1.0" />
+            <xacro:property name="max_torque3" value="3.0" />
             <!-- <xacro:ros2_control_joint_can name="front_left_first_joint" can_id="10" ddq_kp="${kp1}"
                 ddq_kd="${kd1}" max_torque="${max_torque1}" />

Commit message: Kinematics works - PIDs are needed to be tuned
Signed-off-by: Jakub Delicat <delicat.kuba@gmail.com>

File: quadruped_robot_description/urdf/ros2_control.urdf.xacro (robot description, xacro)
@@ -7,5 +7,5 @@
               ddq_kp=1.0  ddq_kd=0.15">
         <joint name="${name}">
-            <command_interface name="acceleration" />
+            <command_interface name="effort" />
             <state_interface name="position">
                 <param name="initial_value">0.0</param>
@@ -75,13 +75,13 @@
             <xacro:property name="kp1" value="25" />
             <xacro:property name="kd1" value="5.0" />
-            <xacro:property name="max_torque1" value="3.0" />
+            <xacro:property name="max_torque1" value="2.0" />
             <!-- <xacro:property name="kp2" value="50" /> -->
             <xacro:property name="kp2" value="7.5" />
             <xacro:property name="kd2" value="1.0" />
-            <xacro:property name="max_torque2" value="3.0" />
+            <xacro:property name="max_torque2" value="1.0" />
             <!-- <xacro:property name="kp3" value="50" /> -->
             <xacro:property name="kp3" value="7.5" />
             <xacro:property name="kd3" value="1.0" />
-            <xacro:property name="max_torque3" value="3.0" />
+            <xacro:property name="max_torque3" value="1.0" />
             <xacro:ros2_control_joint_can name="front_left_first_joint" can_id="10" ddq_kp="${kp1}"
                 ddq_kd="${kd1}" max_torque="${max_torque1}" />
