Commit message: Better pids
Signed-off-by: Jakub Delicat <delicat.kuba@gmail.com>

File: quadruped_robot_description/urdf/quadruped_robot.urdf.xacro (robot description, xacro)
@@ -1,4 +1,5 @@
 <?xml version="1.0"?>
 <robot name="quadruped" xmlns:xacro="http://www.ros.org/wiki/xacro">
+  <xacro:arg name="use_hardware" default="True" />
   <material name="grey">
     <color rgba="0.5 0.5 0.5 1" />
@@ -283,33 +284,40 @@
   <ros2_control name="MD80HardwareInterface" type="system">
     <hardware>
-      <plugin>md80_hardware_interface/MD80HardwareInterface</plugin>
-      <!-- <plugin>mock_components/GenericSystem</plugin> -->
+      <!-- <plugin>md80_hardware_interface/MD80HardwareInterface</plugin> -->
+      <xacro:if value="$(arg use_hardware)">
+        <plugin>md80_hardware_interface/MD80HardwareInterface</plugin>
+      </xacro:if>
+      <xacro:unless value="$(arg use_hardware)">
+        <plugin>mock_components/GenericSystem</plugin>
+      </xacro:unless>
       <param name="encoders_cpr">4096</param>
     </hardware>
-    <xacro:ros2_control_joint_can name="front_left_first_joint" can_id="10" ddq_kp="40.0"
-    ddq_kd="10.0" max_torque="15.0" />
-    <xacro:ros2_control_joint_can name="front_left_second_joint" can_id="11" ddq_kp="20.0"
-    ddq_kd="1.0" />
-    <xacro:ros2_control_joint_can name="front_left_third_joint" can_id="12" ddq_kp="20.0"
-    ddq_kd="1.0" />
-    <xacro:ros2_control_joint_can name="front_right_first_joint" can_id="20" ddq_kp="40.0"
-    ddq_kd="10.0" max_torque="15.0" />
-    <xacro:ros2_control_joint_can name="front_right_second_joint" can_id="21" ddq_kp="20.0"
-    ddq_kd="1.0" />
-    <xacro:ros2_control_joint_can name="front_right_third_joint" can_id="22" ddq_kp="20.0"
-    ddq_kd="1.0" />
-    <xacro:ros2_control_joint_can name="rear_right_first_joint" can_id="30" ddq_kp="40.0"
-    ddq_kd="10.0" max_torque="15.0" />
-    <xacro:ros2_control_joint_can name="rear_right_second_joint" can_id="31" ddq_kp="20.0"
-    ddq_kd="1.0" />
-    <xacro:ros2_control_joint_can name="rear_right_third_joint" can_id="32" ddq_kp="20.0"
+    <xacro:property name="kp2" value="60" />
+    <xacro:property name="kp3" value="20" />
+    <xacro:ros2_control_joint_can name="front_left_first_joint" can_id="10" ddq_kp="80.0"
+    ddq_kd="12.0" max_torque="15.0" />
+    <xacro:ros2_control_joint_can name="front_left_second_joint" can_id="11" ddq_kp="${kp2}"
+    ddq_kd="1.0" />
+    <xacro:ros2_control_joint_can name="front_left_third_joint" can_id="12" ddq_kp="${kp3}"
+    ddq_kd="1.0" />
+    <xacro:ros2_control_joint_can name="front_right_first_joint" can_id="20" ddq_kp="80.0"
+    ddq_kd="12.0" max_torque="15.0" />
+    <xacro:ros2_control_joint_can name="front_right_second_joint" can_id="21" ddq_kp="${kp2}"
+    ddq_kd="1.0" />
+    <xacro:ros2_control_joint_can name="front_right_third_joint" can_id="22" ddq_kp="${kp3}"
+    ddq_kd="1.0" />
+    <xacro:ros2_control_joint_can name="rear_right_first_joint" can_id="30" ddq_kp="80.0"
+    ddq_kd="12.0" max_torque="15.0" />
+    <xacro:ros2_control_joint_can name="rear_right_second_joint" can_id="31" ddq_kp="${kp2}"
+    ddq_kd="1.0" />
+    <xacro:ros2_control_joint_can name="rear_right_third_joint" can_id="32" ddq_kp="${kp3}"
     ddq_kd="1.0" />
     <!-- <xacro:ros2_control_passive_point name="rear_right_fourth_joint" />
     <xacro:ros2_control_passive_point name="rear_right_fifth_joint" /> -->
-    <xacro:ros2_control_joint_can name="rear_left_first_joint" can_id="40" ddq_kp="40.0"
-    ddq_kd="10.0" max_torque="15.0" />
-    <xacro:ros2_control_joint_can name="rear_left_second_joint" can_id="41" ddq_kp="20.0"
+    <xacro:ros2_control_joint_can name="rear_left_first_joint" can_id="40" ddq_kp="80.0"
+    ddq_kd="12.0" max_torque="15.0" />
+    <xacro:ros2_control_joint_can name="rear_left_second_joint" can_id="41" ddq_kp="${kp2}"
       ddq_kd="1.0" />
-    <xacro:ros2_control_joint_can name="rear_left_third_joint" can_id="42" ddq_kp="20.0"
+    <xacro:ros2_control_joint_can name="rear_left_third_joint" can_id="42" ddq_kp="${kp3}"
     ddq_kd="1.0" />
     <!-- <xacro:ros2_control_passive_point name="rear_left_fourth_joint" />

Commit message: Added imu_hw
Signed-off-by: Jakub Delicat <delicat.kuba@gmail.com>

File: quadruped_robot_description/urdf/quadruped_robot.urdf.xacro (robot description, xacro)
@@ -28,4 +28,10 @@
     </inertial>
   </link>
+  <link name="imu_link"/>
+  <joint name="imu_joint" type="fixed">
+    <parent link="base_link" />
+    <child link="imu_link" />
+    <origin xyz="0.0 0.0 0.1" rpy="0.0 0.0 0.0" />
+  </joint>
   <!-- Macro to define a leg -->
   <xacro:macro name="leg"
@@ -293,34 +299,60 @@
       <param name="encoders_cpr">4096</param>
     </hardware>
+    <xacro:property name="kp1" value="80" />
+    <xacro:property name="kd1" value="12" />
     <xacro:property name="kp2" value="60" />
+    <xacro:property name="kd2" value="1" />
     <xacro:property name="kp3" value="20" />
-    <xacro:ros2_control_joint_can name="front_left_first_joint" can_id="10" ddq_kp="80.0"
-    ddq_kd="12.0" max_torque="15.0" />
+    <xacro:property name="kd3" value="1" />
+    <xacro:ros2_control_joint_can name="front_left_first_joint" can_id="10" ddq_kp="${kp1}"
+    ddq_kd="${kd1}" max_torque="15.0" />
     <xacro:ros2_control_joint_can name="front_left_second_joint" can_id="11" ddq_kp="${kp2}"
-    ddq_kd="1.0" />
+    ddq_kd="${kd2}" />
     <xacro:ros2_control_joint_can name="front_left_third_joint" can_id="12" ddq_kp="${kp3}"
-    ddq_kd="1.0" />
-    <xacro:ros2_control_joint_can name="front_right_first_joint" can_id="20" ddq_kp="80.0"
-    ddq_kd="12.0" max_torque="15.0" />
+    ddq_kd="${kd3}" />
+    <xacro:ros2_control_joint_can name="front_right_first_joint" can_id="20" ddq_kp="${kp1}"
+    ddq_kd="${kd1}" max_torque="15.0" />
     <xacro:ros2_control_joint_can name="front_right_second_joint" can_id="21" ddq_kp="${kp2}"
-    ddq_kd="1.0" />
+    ddq_kd="${kd2}" />
     <xacro:ros2_control_joint_can name="front_right_third_joint" can_id="22" ddq_kp="${kp3}"
-    ddq_kd="1.0" />
-    <xacro:ros2_control_joint_can name="rear_right_first_joint" can_id="30" ddq_kp="80.0"
-    ddq_kd="12.0" max_torque="15.0" />
+    ddq_kd="${kd3}" />
+    <xacro:ros2_control_joint_can name="rear_right_first_joint" can_id="30" ddq_kp="${kp1}"
+    ddq_kd="${kd1}" max_torque="15.0" />
     <xacro:ros2_control_joint_can name="rear_right_second_joint" can_id="31" ddq_kp="${kp2}"
-    ddq_kd="1.0" />
+    ddq_kd="${kd2}" />
     <xacro:ros2_control_joint_can name="rear_right_third_joint" can_id="32" ddq_kp="${kp3}"
-    ddq_kd="1.0" />
+    ddq_kd="${kd3}" />
     <!-- <xacro:ros2_control_passive_point name="rear_right_fourth_joint" />
     <xacro:ros2_control_passive_point name="rear_right_fifth_joint" /> -->
-    <xacro:ros2_control_joint_can name="rear_left_first_joint" can_id="40" ddq_kp="80.0"
-    ddq_kd="12.0" max_torque="15.0" />
+    <xacro:ros2_control_joint_can name="rear_left_first_joint" can_id="40" ddq_kp="${kp1}"
+    ddq_kd="${kd1}" max_torque="15.0" />
     <xacro:ros2_control_joint_can name="rear_left_second_joint" can_id="41" ddq_kp="${kp2}"
-      ddq_kd="1.0" />
+      ddq_kd="${kd2}" />
     <xacro:ros2_control_joint_can name="rear_left_third_joint" can_id="42" ddq_kp="${kp3}"
-    ddq_kd="1.0" />
+    ddq_kd="${kd3}" />
     <!-- <xacro:ros2_control_passive_point name="rear_left_fourth_joint" />
     <xacro:ros2_control_passive_point name="rear_left_fifth_joint" /> -->
   </ros2_control>
+  <ros2_control name="imu" type="sensor">
+    <hardware>
+      <plugin>bmx160_serial_hardware_interface/BMX160SerialHardwareInterface</plugin>
+      <param name="port">/dev/ttyACM1</param>
+      <param name="baud_rate">9600</param>
+    </hardware>
+    <sensor name="imu">
+      <!-- <state_interface name="orientation.x" />
+      <state_interface name="orientation.y" />
+      <state_interface name="orientation.z" />
+      <state_interface name="orientation.w" /> -->
+      <state_interface name="magnetometer.x" />
+      <state_interface name="magnetometer.y" />
+      <state_interface name="magnetometer.z" />
+      <state_interface name="angular_velocity.x" />
+      <state_interface name="angular_velocity.y" />
+      <state_interface name="angular_velocity.z" />
+      <state_interface name="linear_acceleration.x" />
+      <state_interface name="linear_acceleration.y" />
+      <state_interface name="linear_acceleration.z" />
+    </sensor>
+  </ros2_control>
 </robot>
