Commit message: Walking robot
Signed-off-by: Jakub Delicat <delicat.kuba@gmail.com>

File: quadruped_robot_description/urdf/quadruped_robot.urdf.xacro (robot description, xacro)
@@ -1,4 +1,6 @@
 <?xml version="1.0"?>
 <robot name="quadruped" xmlns:xacro="http://www.ros.org/wiki/xacro">
+  <xacro:include filename="$(find quadruped_robot_description)/urdf/leg.urdf.xacro" />
+  <xacro:include filename="$(find quadruped_robot_description)/urdf/ros2_control.urdf.xacro" />
   <xacro:arg name="use_hardware" default="True" />
   <material name="grey">
@@ -28,5 +30,5 @@
     </inertial>
   </link>
-  <link name="imu_link"/>
+  <link name="imu_link" />
   <joint name="imu_joint" type="fixed">
     <parent link="base_link" />
@@ -34,335 +36,14 @@
     <origin xyz="0.0 0.0 0.1" rpy="0.0 0.0 0.0" />
   </joint>
-  <!-- Macro to define a leg -->
-  <xacro:macro name="leg"
-    params="prefix xyz rpy first_x:=0.1 first_joint_offset second_joint_offset ">
-    <xacro:property name="zero_angle_offset" value="0.17692153346630435" />
-    <!-- Define the thigh -->
-    <link name="${prefix}_leg_base_link" />
-    <!-- Define the joints -->
-    <joint
-      name="${prefix}_base_to_leg_joint" type="fixed">
-      <parent link="base_link" />
-      <child link="${prefix}_leg_base_link" />
-      <origin xyz="${xyz}" rpy="${rpy}" />
-    </joint>
-    <xacro:first_link
-      name="${prefix}_first_link" />
-    <joint
-      name="${prefix}_leg_base_to_first_link_joint" type="fixed">
-      <parent link="${prefix}_leg_base_link" />
-      <child link="${prefix}_first_link" />
-      <origin xyz="0.0 0.0 0.0" rpy="${-pi/2.0} 0.0 0.0" />
-    </joint>
-    <xacro:second_link
-      name="${prefix}_second_link" />
-    <joint name="${prefix}_first_joint"
-      type="revolute">
-      <parent link="${prefix}_first_link" />
-      <child link="${prefix}_second_link" />
-      <origin xyz="0.031 0.0 0.0" rpy="${first_joint_offset} 0.0 0.0" />
-      <axis xyz="1 0 0" />
-      <limit lower="-3.1416" upper="3.1416" effort="100" velocity="0.5" />
-    </joint>
-    <xacro:third_link
-      name="${prefix}_third_link" />
-    <joint name="${prefix}_second_joint"
-      type="revolute">
-      <parent link="${prefix}_second_link" />
-      <child link="${prefix}_third_link" />
-      <origin xyz="0.064 0.0 0.023" rpy="0.0 0.0 ${second_joint_offset} " />
-      <axis xyz="0 0 1" />
-      <limit lower="-3.14" upper="3.14" effort="100" velocity="0.5" />
-      <dynamics damping="0" friction="0" />
-    </joint>
-    <xacro:fourth_link
-      name="${prefix}_fourth_link" />
-    <joint name="${prefix}_third_joint"
-      type="revolute">
-      <parent link="${prefix}_third_link" />
-      <child link="${prefix}_fourth_link" />
-      <origin xyz="0.0 0.0 0.0555" rpy="0.0 0.0 0.0" />
-      <axis xyz="0 0 1" />
-      <limit lower="-3.14" upper="3.14" effort="100" velocity="0.5" />
-      <dynamics damping="0" friction="0" />
-    </joint>
-    <xacro:fifth_link
-      name="${prefix}_fifth_link" />
-    <joint name="${prefix}_forth_joint"
-      type="continuous">
-      <parent link="${prefix}_fourth_link" />
-      <child link="${prefix}_fifth_link" />
-      <origin xyz="0.125 0.0 0.0255" rpy="0.0 0.0 ${pi}" />
-      <axis xyz="0 0 -1" />
-      <limit lower="-3.14" upper="3.14" effort="100" velocity="0.5" />
-      <dynamics damping="0" friction="0" />
-    </joint>
-    <xacro:sixth_link
-      name="${prefix}_sixth_link" />
-    <joint name="${prefix}_fifth_joint"
-      type="continuous">
-      <parent link="${prefix}_third_link" />
-      <child link="${prefix}_sixth_link" />
-      <origin xyz="-0.125 0.0 0.058" rpy="0.0 0.0 0.0" />
-      <axis xyz="0 0 -1" />
-      <limit lower="-3.14" upper="3.14" effort="100" velocity="0.5" />
-      <dynamics damping="0" friction="0" />
-    </joint>
-  </xacro:macro>
-  <xacro:macro name="first_link" params="name">
-    <link name="${name}">
-      <visual>
-        <origin rpy="0 0 0" xyz="0.0 0 0.0" />
-        <geometry>
-          <mesh filename="package://quadruped_robot_description/meshes/first_link.dae" />
-        </geometry>
-      </visual>
-      <collision>
-        <origin rpy="0 0 0" xyz="0.0 0 0.0" />
-        <geometry>
-          <mesh filename="package://quadruped_robot_description/meshes/first_link.dae" />
-        </geometry>
-      </collision>
-      <inertial>
-        <mass value="0.5" />
-        <origin xyz="0 0 -0.2" />
-        <inertia ixx="0.05" ixy="0.0" ixz="0.0" iyy="0.05" iyz="0.0" izz="0.05" />
-      </inertial>
-    </link>
-  </xacro:macro>
-  <xacro:macro name="second_link" params="name">
-    <link name="${name}">
-      <visual>
-        <origin rpy="0 0 0" xyz="0.0 0 0.0" />
-        <geometry>
-          <mesh filename="package://quadruped_robot_description/meshes/second_link.dae" />
-        </geometry>
-      </visual>
-      <collision>
-        <origin rpy="0 0 0" xyz="0.0 0 0.0" />
-        <geometry>
-          <mesh filename="package://quadruped_robot_description/meshes/second_link.dae" />
-        </geometry>
-      </collision>
-      <inertial>
-        <mass value="0.5" />
-        <origin xyz="0 0 -0.2" />
-        <inertia ixx="0.05" ixy="0.0" ixz="0.0" iyy="0.05" iyz="0.0" izz="0.05" />
-      </inertial>
-    </link>
-  </xacro:macro>
-  <xacro:macro name="third_link" params="name">
-    <link name="${name}">
-      <visual>
-        <origin rpy="0 0 0" xyz="0.0 0 0.0" />
-        <geometry>
-          <mesh filename="package://quadruped_robot_description/meshes/third_link.dae" />
-        </geometry>
-      </visual>
-      <collision>
-        <origin rpy="0 0 0" xyz="0.0 0 0.0" />
-        <geometry>
-          <mesh filename="package://quadruped_robot_description/meshes/third_link.dae" />
-        </geometry>
-      </collision>
-      <inertial>
-        <mass value="0.5" />
-        <origin xyz="0 0 -0.2" />
-        <inertia ixx="0.05" ixy="0.0" ixz="0.0" iyy="0.05" iyz="0.0" izz="0.05" />
-      </inertial>
-    </link>
-  </xacro:macro>
-  <xacro:macro name="fourth_link" params="name">
-    <link name="${name}">
-      <visual>
-        <origin rpy="0 0 0" xyz="0.0 0 0.0" />
-        <geometry>
-          <mesh filename="package://quadruped_robot_description/meshes/fourth_link.dae" />
-        </geometry>
-      </visual>
-      <collision>
-        <origin rpy="0 0 0" xyz="0.0 0 0.0" />
-        <geometry>
-          <mesh filename="package://quadruped_robot_description/meshes/third_link.dae" />
-        </geometry>
-      </collision>
-      <inertial>
-        <mass value="0.5" />
-        <origin xyz="0 0 -0.2" />
-        <inertia ixx="0.05" ixy="0.0" ixz="0.0" iyy="0.05" iyz="0.0" izz="0.05" />
-      </inertial>
-    </link>
-  </xacro:macro>
-  <xacro:macro name="fifth_link" params="name">
-    <link name="${name}">
-      <visual>
-        <origin rpy="0 0 0" xyz="0.0 0 0.0" />
-        <geometry>
-          <mesh filename="package://quadruped_robot_description/meshes/fifth_link.dae" />
-        </geometry>
-      </visual>
-      <collision>
-        <origin rpy="0 0 0" xyz="0.0 0 0.0" />
-        <geometry>
-          <mesh filename="package://quadruped_robot_description/meshes/fifth_link.dae" />
-        </geometry>
-      </collision>
-      <inertial>
-        <mass value="0.5" />
-        <origin xyz="0 0 -0.2" />
-        <inertia ixx="0.05" ixy="0.0" ixz="0.0" iyy="0.05" iyz="0.0" izz="0.05" />
-      </inertial>
-    </link>
-  </xacro:macro>
-  <xacro:macro name="sixth_link" params="name">
-    <link name="${name}">
-      <visual>
-        <origin rpy="0 0 0" xyz="0.0 0 0.0" />
-        <geometry>
-          <mesh filename="package://quadruped_robot_description/meshes/sixth_link.dae" />
-        </geometry>
-      </visual>
-      <collision>
-        <origin rpy="0 0 0" xyz="0.0 0 0.0" />
-        <geometry>
-          <mesh filename="package://quadruped_robot_description/meshes/sixth_link.dae" />
-        </geometry>
-      </collision>
-      <inertial>
-        <mass value="0.5" />
-        <origin xyz="0 0 -0.2" />
-        <inertia ixx="0.05" ixy="0.0" ixz="0.0" iyy="0.05" iyz="0.0" izz="0.05" />
-      </inertial>
-    </link>
-  </xacro:macro>
-  <link name="front_left_leg_deltoid"></link>
-  <joint name="front_left_leg_deltoid_joint" type="fixed">
-    <parent link="front_left_leg_base_link" />
-    <child link="front_left_leg_deltoid" />
-    <origin xyz="${0.031 + 0.068} ${0.023 + 0.0555} 0.0" rpy="${-pi/2.0} 0.0 0.0" />
-  </joint>
   <!-- Define the four legs -->
   <xacro:leg prefix="rear_left" xyz="-0.131 0.06 0.06" rpy="0 0 ${pi}" first_joint_offset="${pi}"
-    second_joint_offset="${pi}" />
+    third_joint_gear_correction_dir="-1.0" />
   <xacro:leg prefix="rear_right" xyz="-0.131 -0.06 0.06" rpy="0 0 ${pi}" first_joint_offset="0.0"
-    second_joint_offset="${pi}" />
+    third_joint_gear_correction_dir="1.0" />
   <xacro:leg prefix="front_right" xyz="0.131 -0.06 0.06" rpy="0 0 0" first_joint_offset="${pi}"
-    second_joint_offset="${pi}" />
+    third_joint_gear_correction_dir="-1.0" />
   <xacro:leg prefix="front_left" xyz="0.131 0.06 0.06" rpy="0 0 0" first_joint_offset="0.0"
-    second_joint_offset="${pi}"
+    third_joint_gear_correction_dir="1.0"
   />
-  <xacro:macro name="ros2_control_joint_can"
-    params="name can_id max_torque=15.0
-              q_kp=10.0   q_ki=0.5    q_kd=0.0    q_windup=1.0
-              dq_kp=2.0   dq_ki=0.5   dq_kd=0.0   dq_windup=0.1
-              ddq_kp=1.0  ddq_kd=0.15">
-    <joint name="${name}">
-      <command_interface name="position" />
-      <state_interface name="position" />
-      <state_interface name="velocity">
-        <param name="initial_value">0.0</param>
-      </state_interface>
-      <state_interface name="effort" />
-      <param name="can_id">${can_id}</param>
-      <param name="max_torque">${max_torque}</param>
-      <param name="q_kp">${q_kp}</param>
-      <param name="q_ki">${q_ki}</param>
-      <param name="q_kd">${q_kd}</param>
-      <param name="q_windup">${q_windup}</param>
-      <param name="dq_kp">${dq_kp}</param>
-      <param name="dq_ki">${dq_ki}</param>
-      <param name="dq_kd">${dq_kd}</param>
-      <param name="dq_windup">${dq_windup}</param>
-      <param name="ddq_kp">${ddq_kp}</param>
-      <param name="ddq_kd">${ddq_kd}</param>
-    </joint>
-  </xacro:macro>
-  <xacro:macro name="ros2_control_passive_point" params="name">
-    <joint name="${name}">
-      <state_interface name="position" />
-      <!-- TODO @delipl
-       <state_interface name="velocity">
-        <param name="initial_value">0.0</param>
-      </state_interface> -->
-      <!-- <state_interface name="effort" /> -->
-    </joint>
-  </xacro:macro>
-  <ros2_control name="MD80HardwareInterface" type="system">
-    <hardware>
-      <!-- <plugin>md80_hardware_interface/MD80HardwareInterface</plugin> -->
-      <xacro:if value="$(arg use_hardware)">
-        <plugin>md80_hardware_interface/MD80HardwareInterface</plugin>
-      </xacro:if>
-      <xacro:unless value="$(arg use_hardware)">
-        <plugin>mock_components/GenericSystem</plugin>
-      </xacro:unless>
-      <param name="encoders_cpr">4096</param>
-    </hardware>
-    <xacro:property name="kp1" value="80" />
-    <xacro:property name="kd1" value="12" />
-    <xacro:property name="kp2" value="60" />
-    <xacro:property name="kd2" value="1" />
-    <xacro:property name="kp3" value="20" />
-    <xacro:property name="kd3" value="1" />
-    <xacro:ros2_control_joint_can name="front_left_first_joint" can_id="10" ddq_kp="${kp1}"
-    ddq_kd="${kd1}" max_torque="15.0" />
-    <xacro:ros2_control_joint_can name="front_left_second_joint" can_id="11" ddq_kp="${kp2}"
-    ddq_kd="${kd2}" />
-    <xacro:ros2_control_joint_can name="front_left_third_joint" can_id="12" ddq_kp="${kp3}"
-    ddq_kd="${kd3}" />
-    <xacro:ros2_control_joint_can name="front_right_first_joint" can_id="20" ddq_kp="${kp1}"
-    ddq_kd="${kd1}" max_torque="15.0" />
-    <xacro:ros2_control_joint_can name="front_right_second_joint" can_id="21" ddq_kp="${kp2}"
-    ddq_kd="${kd2}" />
-    <xacro:ros2_control_joint_can name="front_right_third_joint" can_id="22" ddq_kp="${kp3}"
-    ddq_kd="${kd3}" />
-    <xacro:ros2_control_joint_can name="rear_right_first_joint" can_id="30" ddq_kp="${kp1}"
-    ddq_kd="${kd1}" max_torque="15.0" />
-    <xacro:ros2_control_joint_can name="rear_right_second_joint" can_id="31" ddq_kp="${kp2}"
-    ddq_kd="${kd2}" />
-    <xacro:ros2_control_joint_can name="rear_right_third_joint" can_id="32" ddq_kp="${kp3}"
-    ddq_kd="${kd3}" />
-    <!-- <xacro:ros2_control_passive_point name="rear_right_fourth_joint" />
-    <xacro:ros2_control_passive_point name="rear_right_fifth_joint" /> -->
-    <xacro:ros2_control_joint_can name="rear_left_first_joint" can_id="40" ddq_kp="${kp1}"
-    ddq_kd="${kd1}" max_torque="15.0" />
-    <xacro:ros2_control_joint_can name="rear_left_second_joint" can_id="41" ddq_kp="${kp2}"
-      ddq_kd="${kd2}" />
-    <xacro:ros2_control_joint_can name="rear_left_third_joint" can_id="42" ddq_kp="${kp3}"
-    ddq_kd="${kd3}" />
-    <!-- <xacro:ros2_control_passive_point name="rear_left_fourth_joint" />
-    <xacro:ros2_control_passive_point name="rear_left_fifth_joint" /> -->
-  </ros2_control>
-  <ros2_control name="imu" type="sensor">
-    <hardware>
-      <plugin>bmx160_serial_hardware_interface/BMX160SerialHardwareInterface</plugin>
-      <param name="port">/dev/ttyACM1</param>
-      <param name="baud_rate">9600</param>
-      <!-- Madgwick Filter Params -->
-      <!-- https://www.mouser.com/pdfdocs/BST-BMX160-DS000-11.pdf -->
-      <!-- Output Noise 0.007 -->
-      <!-- Bias stability 0.0000145 -->
-      <param name="gain">0.003031089</param>
-      <param name="zeta">0.000006279</param>
-      <param name="mag_bias_x">0.002</param>
-      <param name="mag_bias_y">0.002</param>
-      <param name="mag_bias_z">0.002</param>
-      <param name="world_frame">enu</param>
-    </hardware>
-    <sensor name="imu">
-      <!-- <state_interface name="orientation.x" />
-      <state_interface name="orientation.y" />
-      <state_interface name="orientation.z" />
-      <state_interface name="orientation.w" /> -->
-      <state_interface name="magnetometer.x" />
-      <state_interface name="magnetometer.y" />
-      <state_interface name="magnetometer.z" />
-      <state_interface name="angular_velocity.x" />
-      <state_interface name="angular_velocity.y" />
-      <state_interface name="angular_velocity.z" />
-      <state_interface name="linear_acceleration.x" />
-      <state_interface name="linear_acceleration.y" />
-      <state_interface name="linear_acceleration.z" />
-    </sensor>
-  </ros2_control>
+  <xacro:quadruperd_ros2_control use_hardware="$(arg use_hardware)" />
 </robot>

Commit message: IMU fake
Signed-off-by: Jakub Delicat <delicat.kuba@gmail.com>

File: quadruped_robot_description/urdf/quadruped_robot.urdf.xacro (robot description, xacro)
@@ -34,5 +34,5 @@
     <parent link="base_link" />
     <child link="imu_link" />
-    <origin xyz="0.0 0.0 0.1" rpy="0.0 0.0 0.0" />
+    <origin xyz="0.0 0.0 0.1" rpy=" 0.0 ${pi} 0.0" />
   </joint>
   <!-- Define the four legs -->

File: quadruped_robot_description/urdf/ros2_control.urdf.xacro (robot description, xacro)
@@ -47,4 +47,5 @@
                     <plugin>md80_hardware_interface/MD80HardwareInterface</plugin>
                     <param name="usb_port">/dev/ttyACM0</param>
+                    <param name="bus">spi</param>
                 </xacro:if>
                 <xacro:unless value="${use_hardware}">
@@ -57,26 +58,28 @@
             <xacro:property name="kp2" value="50" />
             <xacro:property name="kd2" value="10" />
+            <xacro:property name="max_torque2" value="10.0" />
             <!-- <xacro:property name="kp3" value="50" /> -->
-            <xacro:property name="kp3" value="25" />
+            <xacro:property name="kp3" value="50" />
             <xacro:property name="kd3" value="10" />
+            <xacro:property name="max_torque3" value="10.0" />
             <xacro:ros2_control_joint_can name="front_left_first_joint" can_id="10" ddq_kp="${kp1}"
                 ddq_kd="${kd1}" max_torque="15.0" />
             <xacro:ros2_control_joint_can name="front_left_second_joint" can_id="11" ddq_kp="${kp2}"
-                ddq_kd="${kd2}" />
+                ddq_kd="${kd2}" max_torque="${max_torque2}" />
             <xacro:ros2_control_joint_can name="front_left_third_joint" can_id="12" ddq_kp="${kp3}"
-                ddq_kd="${kd3}" />
+                ddq_kd="${kd3}" max_torque="${max_torque3}" />
             <xacro:ros2_control_joint_can name="front_right_first_joint" can_id="20" ddq_kp="${kp1}"
                 ddq_kd="${kd1}" max_torque="15.0" />
             <xacro:ros2_control_joint_can name="front_right_second_joint" can_id="21"
                 ddq_kp="${kp2}"
-                ddq_kd="${kd2}" />
+                ddq_kd="${kd2}" max_torque="${max_torque2}" />
             <xacro:ros2_control_joint_can name="front_right_third_joint" can_id="22" ddq_kp="${kp3}"
-                ddq_kd="${kd3}" />
+                ddq_kd="${kd3}" max_torque="${max_torque3}"/>
             <xacro:ros2_control_joint_can name="rear_right_first_joint" can_id="30" ddq_kp="${kp1}"
                 ddq_kd="${kd1}" max_torque="15.0" />
             <xacro:ros2_control_joint_can name="rear_right_second_joint" can_id="31" ddq_kp="${kp2}"
-                ddq_kd="${kd2}" />
+                ddq_kd="${kd2}" max_torque="${max_torque2}"/>
             <xacro:ros2_control_joint_can name="rear_right_third_joint" can_id="32" ddq_kp="${kp3}"
-                ddq_kd="${kd3}" />
+                ddq_kd="${kd3}" max_torque="${max_torque3}"/>
             <!-- <xacro:ros2_control_passive_point name="rear_right_fourth_joint" />
     <xacro:ros2_control_passive_point name="rear_right_fifth_joint" /> -->
@@ -84,7 +87,7 @@
                 ddq_kd="${kd1}" max_torque="15.0" />
             <xacro:ros2_control_joint_can name="rear_left_second_joint" can_id="41" ddq_kp="${kp2}"
-                ddq_kd="${kd2}" />
+                ddq_kd="${kd2}"  max_torque="${max_torque2}" />
             <xacro:ros2_control_joint_can name="rear_left_third_joint" can_id="42" ddq_kp="${kp3}"
-                ddq_kd="${kd3}" />
+                ddq_kd="${kd3}" max_torque="${max_torque3}" />
             <!-- <xacro:ros2_control_passive_point name="rear_left_fourth_joint" />
     <xacro:ros2_control_passive_point name="rear_left_fifth_joint" /> -->
@@ -94,4 +97,41 @@
             <xacro:property name="mock_imu" value="system" />
         </xacro:unless>
+        <ros2_control name="imu" type="${mock_imu}">
+            <hardware>
+                <xacro:if value="${use_hardware}">
+                    <plugin>bmx160_serial_hardware_interface/BMX160SerialHardwareInterface</plugin>
+                </xacro:if>
+                <xacro:unless value="${use_hardware}">
+                    <plugin>mock_components/GenericSystem</plugin>
+                </xacro:unless>
+                <param name="port">/dev/ttyACM0</param>
+                <param name="baud_rate">9600</param>
+                <!-- Madgwick Filter Params -->
+                <!-- https://www.mouser.com/pdfdocs/BST-BMX160-DS000-11.pdf -->
+                <!-- Output Noise 0.007 -->
+                <!-- Bias stability 0.0000145 -->
+                <param name="gain">0.003031089</param>
+                <param name="zeta">0.000006279</param>
+                <param name="mag_bias_x">0.002</param>
+                <param name="mag_bias_y">0.002</param>
+                <param name="mag_bias_z">0.002</param>
+                <param name="world_frame">enu</param>
+            </hardware>
+            <sensor name="imu">
+                <state_interface name="orientation.x" />
+                <state_interface name="orientation.y" />
+                <state_interface name="orientation.z" />
+                <state_interface name="orientation.w" />
+                <state_interface name="magnetometer.x" />
+                <state_interface name="magnetometer.y" />
+                <state_interface name="magnetometer.z" />
+                <state_interface name="angular_velocity.x" />
+                <state_interface name="angular_velocity.y" />
+                <state_interface name="angular_velocity.z" />
+                <state_interface name="linear_acceleration.x" />
+                <state_interface name="linear_acceleration.y" />
+                <state_interface name="linear_acceleration.z" />
+            </sensor>
+        </ros2_control>
     </xacro:macro>
 </robot>

Commit message: Run pre commit | clean up | created four bar bot
Signed-off-by: Jakub Delicat <delicat.kuba@gmail.com>

File: quadruped_robot_description/urdf/quadruped_robot.urdf.xacro (robot description, xacro)
@@ -1,10 +1,11 @@
 <?xml version="1.0"?>
 <robot name="quadruped" xmlns:xacro="http://www.ros.org/wiki/xacro">
-  <xacro:include filename="$(find quadruped_robot_description)/urdf/inertia.urdf.xacro"  />
+  <xacro:include filename="$(find quadruped_robot_description)/urdf/inertia.urdf.xacro" />
   <xacro:include filename="$(find quadruped_robot_description)/urdf/leg.urdf.xacro" />
   <xacro:include filename="$(find quadruped_robot_description)/urdf/ros2_control.urdf.xacro" />
-  <xacro:include filename="$(find quadruped_robot_description)/urdf/gazebo.urdf.xacro"  />
+  <xacro:include filename="$(find quadruped_robot_description)/urdf/gazebo.urdf.xacro" />
   <mujoco>
-    <compiler meshdir="$(find quadruped_robot_description)/meshes" balanceinertia="true" discardvisual="false"/>
+    <compiler meshdir="$(find quadruped_robot_description)/meshes" balanceinertia="true"
+      discardvisual="false" />
   </mujoco>
   <xacro:arg name="use_hardware" default="True" />
@@ -13,5 +14,6 @@
     <color rgba="0.5 0.5 0.5 1" />
   </material>
-  <link name="base_link">
+  <link name="base_link" />
+  <link name="body_link">
     <visual>
       <origin rpy="0 0 ${pi}" xyz="0.0 0 0" />
@@ -29,4 +31,9 @@
     <xacro:box_inertia m="50.0" w="0.59" h="0.225" d="0.1" xyz="0.01 0 0.06" />
   </link>
+  <joint name="body_to_base_joint" type="fixed">
+    <parent link="base_link" />
+    <child link="body_link" />
+    <origin xyz="0.0 0.0 0.0" rpy="0.0 0.0 0.0" />
+  </joint>
   <link name="imu_link" />
   <joint name="imu_joint" type="fixed">
