Commit message: good angles
Signed-off-by: Jakub Delicat <delicat.kuba@gmail.com>

File: mujoco_ros2_control/mujoco_ros2_control_demos/urdf/quadruped_to_mujoco.urdf (robot description, URDF)
Before this commit: robot quadruped, 42 links, 41 joints
Links:
- removed link front_right_chain_close_a_link
- removed link front_right_chain_close_b_link
- removed link front_right_fifth_link
- removed link front_right_first_link
- removed link front_right_foot_link
- removed link front_right_fourth_link
- removed link front_right_leg_base_link
- removed link front_right_second_link
- removed link front_right_sixth_link
- removed link front_right_third_link
- removed link rear_left_chain_close_a_link
- removed link rear_left_chain_close_b_link
- removed link rear_left_fifth_link
- removed link rear_left_first_link
- removed link rear_left_foot_link
- removed link rear_left_fourth_link
- removed link rear_left_leg_base_link
- removed link rear_left_second_link
- removed link rear_left_sixth_link
- removed link rear_left_third_link
- removed link rear_right_chain_close_a_link
- removed link rear_right_chain_close_b_link
- removed link rear_right_fifth_link
- removed link rear_right_first_link
- removed link rear_right_foot_link
- removed link rear_right_fourth_link
- removed link rear_right_leg_base_link
- removed link rear_right_second_link
- removed link rear_right_sixth_link
- removed link rear_right_third_link
Joints:
- removed joint front_left_forth_joint
- removed joint front_right_base_to_leg_joint
- removed joint front_right_chain_close_a_joint
- removed joint front_right_chain_close_b_joint
- removed joint front_right_fifth_joint
- removed joint front_right_first_joint
- removed joint front_right_foot_joint
- removed joint front_right_forth_joint
- removed joint front_right_leg_base_to_first_link_joint
- removed joint front_right_second_joint
- removed joint front_right_third_joint
- removed joint rear_left_base_to_leg_joint
- removed joint rear_left_chain_close_a_joint
- removed joint rear_left_chain_close_b_joint
- removed joint rear_left_fifth_joint
- removed joint rear_left_first_joint
- removed joint rear_left_foot_joint
- removed joint rear_left_forth_joint
- removed joint rear_left_leg_base_to_first_link_joint
- removed joint rear_left_second_joint
- removed joint rear_left_third_joint
- removed joint rear_right_base_to_leg_joint
- removed joint rear_right_chain_close_a_joint
- removed joint rear_right_chain_close_b_joint
- removed joint rear_right_fifth_joint
- removed joint rear_right_first_joint
- removed joint rear_right_foot_joint
- removed joint rear_right_forth_joint
- removed joint rear_right_leg_base_to_first_link_joint
- removed joint rear_right_second_joint
- removed joint rear_right_third_joint
- added joint front_left_fourth_joint: type revolute, parent front_left_fourth_link, child front_left_fifth_link, origin xyz=0.125 0.0 0.0255 rpy=0.0 0.0 3.141592653589793, axis 0 0 -1, limit lower=-0.8 upper=-2.9 effort=  2.0 velocity=0.1

Commit message: Standing up in mujoco
Signed-off-by: Jakub Delicat <delicat.kuba@gmail.com>

File: mujoco_ros2_control/mujoco_ros2_control_demos/urdf/quadruped_to_mujoco.urdf (robot description, URDF)
Before this commit: robot quadruped, 42 links, 41 joints
Joints:
- joint front_left_second_joint: limit lower=1.57 upper=4.71 effort=100.0 velocity=0.1 -> lower=-3.14 upper=3.14 effort=100.0 velocity=0.1
- joint front_left_third_joint: axis 0 0 1 -> 0 0 -1
- joint front_right_second_joint: axis 0 0 1 -> 0 0 -1; limit lower=0 upper=4.71 effort=100.0 velocity=0.1 -> lower=-3.14 upper=3.14 effort=100.0 velocity=0.1
- joint rear_left_second_joint: axis 0 0 1 -> 0 0 -1; limit lower=0.0 upper=4.71 effort=100.0 velocity=0.1 -> lower=-3.14 upper=3.14 effort=100.0 velocity=0.1
- joint rear_right_second_joint: limit lower=1.57 upper=4.71 effort=100.0 velocity=0.1 -> lower=-3.14 upper=3.14 effort=100.0 velocity=0.1
- joint rear_right_third_joint: axis 0 0 1 -> 0 0 -1
