Commit message: standing robot
Signed-off-by: Jakub Delicat <delicat.kuba@gmail.com>

File: mujoco_ros2_control/mujoco_ros2_control_demos/urdf/one_leg.urdf (robot description, URDF)
Before this commit: robot quadruped, 42 links, 41 joints
Links:
- removed link front_right_chain_close_a_link
- removed link front_right_chain_close_b_link
- removed link front_right_fifth_link
- removed link front_right_first_link
- removed link front_right_foot_link
- removed link front_right_fourth_link
- removed link front_right_leg_base_link
- removed link front_right_second_link
- removed link front_right_sixth_link
- removed link front_right_third_link
- removed link rear_left_chain_close_a_link
- removed link rear_left_chain_close_b_link
- removed link rear_left_fifth_link
- removed link rear_left_first_link
- removed link rear_left_foot_link
- removed link rear_left_fourth_link
- removed link rear_left_leg_base_link
- removed link rear_left_second_link
- removed link rear_left_sixth_link
- removed link rear_left_third_link
- removed link rear_right_chain_close_a_link
- removed link rear_right_chain_close_b_link
- removed link rear_right_fifth_link
- removed link rear_right_first_link
- removed link rear_right_foot_link
- removed link rear_right_fourth_link
- removed link rear_right_leg_base_link
- removed link rear_right_second_link
- removed link rear_right_sixth_link
- removed link rear_right_third_link
Joints:
- removed joint front_right_base_to_leg_joint
- removed joint front_right_chain_close_a_joint
- removed joint front_right_chain_close_b_joint
- removed joint front_right_fifth_joint
- removed joint front_right_first_joint
- removed joint front_right_foot_joint
- removed joint front_right_fourth_joint
- removed joint front_right_leg_base_to_first_link_joint
- removed joint front_right_second_joint
- removed joint front_right_third_joint
- removed joint rear_left_base_to_leg_joint
- removed joint rear_left_chain_close_a_joint
- removed joint rear_left_chain_close_b_joint
- removed joint rear_left_fifth_joint
- removed joint rear_left_first_joint
- removed joint rear_left_foot_joint
- removed joint rear_left_fourth_joint
- removed joint rear_left_leg_base_to_first_link_joint
- removed joint rear_left_second_joint
- removed joint rear_left_third_joint
- removed joint rear_right_base_to_leg_joint
- removed joint rear_right_chain_close_a_joint
- removed joint rear_right_chain_close_b_joint
- removed joint rear_right_fifth_joint
- removed joint rear_right_first_joint
- removed joint rear_right_foot_joint
- removed joint rear_right_fourth_joint
- removed joint rear_right_leg_base_to_first_link_joint
- removed joint rear_right_second_joint
- removed joint rear_right_third_joint

File: mujoco_ros2_control/mujoco_ros2_control_demos/urdf/quadruped_to_pinicchio.urdf (robot description, URDF)
Before this commit: robot quadruped, 42 links, 41 joints
Links:
- removed link front_right_chain_close_a_link
- removed link front_right_chain_close_b_link
- removed link front_right_fifth_link
- removed link front_right_first_link
- removed link front_right_foot_link
- removed link front_right_fourth_link
- removed link front_right_leg_base_link
- removed link front_right_second_link
- removed link front_right_sixth_link
- removed link front_right_third_link
- removed link rear_left_chain_close_a_link
- removed link rear_left_chain_close_b_link
- removed link rear_left_fifth_link
- removed link rear_left_first_link
- removed link rear_left_foot_link
- removed link rear_left_fourth_link
- removed link rear_left_leg_base_link
- removed link rear_left_second_link
- removed link rear_left_sixth_link
- removed link rear_left_third_link
- removed link rear_right_chain_close_a_link
- removed link rear_right_chain_close_b_link
- removed link rear_right_fifth_link
- removed link rear_right_first_link
- removed link rear_right_foot_link
- removed link rear_right_fourth_link
- removed link rear_right_leg_base_link
- removed link rear_right_second_link
- removed link rear_right_sixth_link
- removed link rear_right_third_link
- link base_link: geometry collision mesh filename=/home/rabin/Documents/quadruped_robot/src/quadruped_robot_d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; visual mesh filename=/home/rabin/Documents/quadruped_robot/src/quadruped_robot_d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
- link front_left_fifth_link: geometry collision mesh filename=/home/rabin/Documents/quadruped_robot/src/quadruped_robot_d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; visual mesh filename=/home/rabin/Documents/quadruped_robot/src/quadruped_robot_d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
- link front_left_first_link: geometry collision mesh filename=/home/rabin/Documents/quadruped_robot/src/quadruped_robot_d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; visual mesh filename=/home/rabin/Documents/quadruped_robot/src/quadruped_robot_d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
- link front_left_fourth_link: geometry collision mesh filename=/home/rabin/Documents/quadruped_robot/src/quadruped_robot_d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; visual mesh filename=/home/rabin/Documents/quadruped_robot/src/quadruped_robot_d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
- link front_left_second_link: geometry collision mesh filename=/home/rabin/Documents/quadruped_robot/src/quadruped_robot_d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; visual mesh filename=/home/rabin/Documents/quadruped_robot/src/quadruped_robot_d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
- link front_left_sixth_link: geometry collision mesh filename=/home/rabin/Documents/quadruped_robot/src/quadruped_robot_d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; visual mesh filename=/home/rabin/Documents/quadruped_robot/src/quadruped_robot_d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
- link front_left_third_link: geometry collision mesh filename=/home/rabin/Documents/quadruped_robot/src/quadruped_robot_d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; visual mesh filename=/home/rabin/Documents/quadruped_robot/src/quadruped_robot_d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
Joints:
- removed joint front_right_base_to_leg_joint
- removed joint front_right_chain_close_a_joint
- removed joint front_right_chain_close_b_joint
- removed joint front_right_fifth_joint
- removed joint front_right_first_joint
- removed joint front_right_foot_joint
- removed joint front_right_fourth_joint
- removed joint front_right_leg_base_to_first_link_joint
- removed joint front_right_second_joint
- removed joint front_right_third_joint
- removed joint rear_left_base_to_leg_joint
- removed joint rear_left_chain_close_a_joint
- removed joint rear_left_chain_close_b_joint
- removed joint rear_left_fifth_joint
- removed joint rear_left_first_joint
- removed joint rear_left_foot_joint
- removed joint rear_left_fourth_joint
- removed joint rear_left_leg_base_to_first_link_joint
- removed joint rear_left_second_joint
- removed joint rear_left_third_joint
- removed joint rear_right_base_to_leg_joint
- removed joint rear_right_chain_close_a_joint
- removed joint rear_right_chain_close_b_joint
- removed joint rear_right_fifth_joint
- removed joint rear_right_first_joint
- removed joint rear_right_foot_joint
- removed joint rear_right_fourth_joint
- removed joint rear_right_leg_base_to_first_link_joint
- removed joint rear_right_second_joint
- removed joint rear_right_third_joint

File: quadruped_robot_description/urdf/ros2_control.urdf.xacro (robot description, xacro)
@@ -84,4 +84,5 @@
             <xacro:property name="kp1" value="25" />
             <xacro:property name="kd1" value="5.0" />
+            <xacro:property name="max_torque1" value="15.0" />
             <!-- <xacro:property name="kp2" value="50" /> -->
             <xacro:property name="kp2" value="7.5" />
@@ -93,5 +94,5 @@
             <xacro:property name="max_torque3" value="10.0" />
             <xacro:ros2_control_joint_can name="front_left_first_joint" can_id="10" ddq_kp="${kp1}"
-                ddq_kd="${kd1}" max_torque="15.0" />
+                ddq_kd="${kd1}" max_torque="${max_torque1}" />
             <xacro:ros2_control_joint_can name="front_left_second_joint" can_id="11" ddq_kp="${kp2}"
                 ddq_kd="${kd2}" max_torque="${max_torque2}" />
@@ -99,5 +100,5 @@
                 ddq_kd="${kd3}" max_torque="${max_torque3}" />
             <xacro:ros2_control_joint_can name="front_right_first_joint" can_id="20" ddq_kp="${kp1}"
-                ddq_kd="${kd1}" max_torque="15.0" />
+                ddq_kd="${kd1}" max_torque="${max_torque1}" />
             <xacro:ros2_control_joint_can name="front_right_second_joint" can_id="21"
                 ddq_kp="${kp2}"
@@ -106,5 +107,5 @@
                 ddq_kd="${kd3}" max_torque="${max_torque3}" />
             <xacro:ros2_control_joint_can name="rear_right_first_joint" can_id="30" ddq_kp="${kp1}"
-                ddq_kd="${kd1}" max_torque="15.0" />
+                ddq_kd="${kd1}" max_torque="${max_torque1}" />
             <xacro:ros2_control_joint_can name="rear_right_second_joint" can_id="31" ddq_kp="${kp2}"
                 ddq_kd="${kd2}" max_torque="${max_torque2}" />
@@ -114,5 +115,5 @@
     <xacro:ros2_control_passive_point name="rear_right_fifth_joint" /> -->
             <xacro:ros2_control_joint_can name="rear_left_first_joint" can_id="40" ddq_kp="${kp1}"
-                ddq_kd="${kd1}" max_torque="15.0" />
+                ddq_kd="${kd1}" max_torque="${max_torque1}" />
             <xacro:ros2_control_joint_can name="rear_left_second_joint" can_id="41" ddq_kp="${kp2}"
                 ddq_kd="${kd2}" max_torque="${max_torque2}" />

Commit message: Cleaned quadruped_controller
Signed-off-by: Jakub Delicat <delicat.kuba@gmail.com>

File: mujoco_ros2_control/mujoco_ros2_control_demos/urdf/one_leg.urdf (robot description, URDF)
Before this commit: robot quadruped, 12 links, 11 joints
Links:
- link base_link: geometry collision mesh filename=package://four_bar_bot_description/meshes/base_link.dae; visual mesh filename=package://four_bar_bot_description/meshes/base_link.dae
- link front_left_fifth_link: geometry collision mesh filename=package://four_bar_bot_description/meshes/fifth_link.dae; visual mesh filename=package://four_bar_bot_description/meshes/fifth_link.dae
- link front_left_first_link: geometry collision mesh filename=package://four_bar_bot_description/meshes/first_link.dae; visual mesh filename=package://four_bar_bot_description/meshes/first_link.dae
- link front_left_fourth_link: geometry collision mesh filename=package://four_bar_bot_description/meshes/fourth_link.dae; visual mesh filename=package://four_bar_bot_description/meshes/fourth_link.dae
- link front_left_second_link: geometry collision mesh filename=package://four_bar_bot_description/meshes/second_link.dae; visual mesh filename=package://four_bar_bot_description/meshes/second_link.dae
- link front_left_sixth_link: geometry collision mesh filename=package://four_bar_bot_description/meshes/sixth_link.dae; visual mesh filename=package://four_bar_bot_description/meshes/sixth_link.dae
- link front_left_third_link: geometry collision mesh filename=package://four_bar_bot_description/meshes/third_link.dae; visual mesh filename=package://four_bar_bot_description/meshes/third_link.dae

File: mujoco_ros2_control/mujoco_ros2_control_demos/urdf/quadruped_to_mujoco.urdf (robot description, URDF)
Before this commit: robot quadruped, 42 links, 41 joints
Links:
- link base_link: geometry collision mesh filename=package://four_bar_bot_description/meshes/base_link.dae; visual mesh filename=package://four_bar_bot_description/meshes/base_link.dae
- link front_left_fifth_link: geometry collision mesh filename=package://four_bar_bot_description/meshes/fifth_link.dae; visual mesh filename=package://four_bar_bot_description/meshes/fifth_link.dae
- link front_left_first_link: geometry collision mesh filename=package://four_bar_bot_description/meshes/first_link.dae; visual mesh filename=package://four_bar_bot_description/meshes/first_link.dae
- link front_left_fourth_link: geometry collision mesh filename=package://four_bar_bot_description/meshes/fourth_link.dae; visual mesh filename=package://four_bar_bot_description/meshes/fourth_link.dae
- link front_left_second_link: geometry collision mesh filename=package://four_bar_bot_description/meshes/second_link.dae; visual mesh filename=package://four_bar_bot_description/meshes/second_link.dae
- link front_left_sixth_link: geometry collision mesh filename=package://four_bar_bot_description/meshes/sixth_link.dae; visual mesh filename=package://four_bar_bot_description/meshes/sixth_link.dae
- link front_left_third_link: geometry collision mesh filename=package://four_bar_bot_description/meshes/third_link.dae; visual mesh filename=package://four_bar_bot_description/meshes/third_link.dae
- link front_right_fifth_link: geometry collision mesh filename=package://four_bar_bot_description/meshes/fifth_link.dae; visual mesh filename=package://four_bar_bot_description/meshes/fifth_link.dae
- link front_right_first_link: geometry collision mesh filename=package://four_bar_bot_description/meshes/first_link.dae; visual mesh filename=package://four_bar_bot_description/meshes/first_link.dae
- link front_right_fourth_link: geometry collision mesh filename=package://four_bar_bot_description/meshes/fourth_link.dae; visual mesh filename=package://four_bar_bot_description/meshes/fourth_link.dae
- link front_right_second_link: geometry collision mesh filename=package://four_bar_bot_description/meshes/second_link.dae; visual mesh filename=package://four_bar_bot_description/meshes/second_link.dae
- link front_right_sixth_link: geometry collision mesh filename=package://four_bar_bot_description/meshes/sixth_link.dae; visual mesh filename=package://four_bar_bot_description/meshes/sixth_link.dae
- link front_right_third_link: geometry collision mesh filename=package://four_bar_bot_description/meshes/third_link.dae; visual mesh filename=package://four_bar_bot_description/meshes/third_link.dae
- link rear_left_fifth_link: geometry collision mesh filename=package://four_bar_bot_description/meshes/fifth_link.dae; visual mesh filename=package://four_bar_bot_description/meshes/fifth_link.dae
- link rear_left_first_link: geometry collision mesh filename=package://four_bar_bot_description/meshes/first_link.dae; visual mesh filename=package://four_bar_bot_description/meshes/first_link.dae
- link rear_left_fourth_link: geometry collision mesh filename=package://four_bar_bot_description/meshes/fourth_link.dae; visual mesh filename=package://four_bar_bot_description/meshes/fourth_link.dae
- link rear_left_second_link: geometry collision mesh filename=package://four_bar_bot_description/meshes/second_link.dae; visual mesh filename=package://four_bar_bot_description/meshes/second_link.dae
- link rear_left_sixth_link: geometry collision mesh filename=package://four_bar_bot_description/meshes/sixth_link.dae; visual mesh filename=package://four_bar_bot_description/meshes/sixth_link.dae
- link rear_left_third_link: geometry collision mesh filename=package://four_bar_bot_description/meshes/third_link.dae; visual mesh filename=package://four_bar_bot_description/meshes/third_link.dae
- link rear_right_fifth_link: geometry collision mesh filename=package://four_bar_bot_description/meshes/fifth_link.dae; visual mesh filename=package://four_bar_bot_description/meshes/fifth_link.dae
- link rear_right_first_link: geometry collision mesh filename=package://four_bar_bot_description/meshes/first_link.dae; visual mesh filename=package://four_bar_bot_description/meshes/first_link.dae
- link rear_right_fourth_link: geometry collision mesh filename=package://four_bar_bot_description/meshes/fourth_link.dae; visual mesh filename=package://four_bar_bot_description/meshes/fourth_link.dae
- link rear_right_second_link: geometry collision mesh filename=package://four_bar_bot_description/meshes/second_link.dae; visual mesh filename=package://four_bar_bot_description/meshes/second_link.dae
- link rear_right_sixth_link: geometry collision mesh filename=package://four_bar_bot_description/meshes/sixth_link.dae; visual mesh filename=package://four_bar_bot_description/meshes/sixth_link.dae
- link rear_right_third_link: geometry collision mesh filename=package://four_bar_bot_description/meshes/third_link.dae; visual mesh filename=package://four_bar_bot_description/meshes/third_link.dae

File: mujoco_ros2_control/mujoco_ros2_control_demos/urdf/quadruped_to_pinicchio.urdf (robot description, URDF)
Before this commit: robot quadruped, 12 links, 11 joints
Links:
- link base_link: geometry collision mesh filename=/home/rabin/Documents/quadruped_robot/src/four_bar_bot_desc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; visual mesh filename=/home/rabin/Documents/quadruped_robot/src/four_bar_bot_desc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
- link front_left_fifth_link: geometry collision mesh filename=/home/rabin/Documents/quadruped_robot/src/four_bar_bot_desc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; visual mesh filename=/home/rabin/Documents/quadruped_robot/src/four_bar_bot_desc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
- link front_left_first_link: geometry collision mesh filename=/home/rabin/Documents/quadruped_robot/src/four_bar_bot_desc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; visual mesh filename=/home/rabin/Documents/quadruped_robot/src/four_bar_bot_desc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
- link front_left_fourth_link: geometry collision mesh filename=/home/rabin/Documents/quadruped_robot/src/four_bar_bot_desc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; visual mesh filename=/home/rabin/Documents/quadruped_robot/src/four_bar_bot_desc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
- link front_left_second_link: geometry collision mesh filename=/home/rabin/Documents/quadruped_robot/src/four_bar_bot_desc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; visual mesh filename=/home/rabin/Documents/quadruped_robot/src/four_bar_bot_desc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
- link front_left_sixth_link: geometry collision mesh filename=/home/rabin/Documents/quadruped_robot/src/four_bar_bot_desc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; visual mesh filename=/home/rabin/Documents/quadruped_robot/src/four_bar_bot_desc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
- link front_left_third_link: geometry collision mesh filename=/home/rabin/Documents/quadruped_robot/src/four_bar_bot_desc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; visual mesh filename=/home/rabin/Documents/quadruped_robot/src/four_bar_bot_desc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
