Commit message: Fixed xacro
Signed-off-by: Jakub Delicat <delicat.kuba@gmail.com>

File: four_bar_bot_description/urdf/leg.urdf.xacro (robot description, xacro)
@@ -39,6 +39,6 @@
     <!-- <xacro:property name="second_joint_gear_correction" value="${third_joint_gear_correction_dir*0.2793}" />
     <xacro:property name="third_joint_gear_correction" value="${-1.117+pi}" /> -->
-    <xacro:property name="second_joint_gear_correction" value="${third_joint_gear_correction_dir*0.2793}" />
-    <xacro:property name="third_joint_gear_correction" value="${-1.117+pi}" />
+    <xacro:property name="second_joint_gear_correction" value="0" />
+    <xacro:property name="third_joint_gear_correction" value="${1.198}" />
     <joint name="${prefix}_second_joint"
       type="revolute">
@@ -46,5 +46,5 @@
       <child link="${prefix}_third_link" />
       <origin xyz="0.064 0.0 0.023"
-        rpy="0.0 0.0 ${pi + second_joint_gear_correction} " />
+        rpy="0.0 0.0 ${pi} " />
       <axis xyz="0 0 1" />
       <limit effort="100.0" lower="1.57" upper="4.71" velocity="10.0" />
@@ -59,5 +59,5 @@
       <origin xyz="0.0 0.0 0.0555"
         rpy="0.0 0.0 ${third_joint_gear_correction_dir*third_joint_gear_correction}" />
-      <axis xyz="0 0 1" />
+      <axis xyz="0 0 ${third_joint_gear_correction_dir}" />
       <limit effort="100.0" lower="0.425" upper="5.8" velocity="10.0" />
       <dynamics damping="0.1" friction="0.1" />
@@ -71,5 +71,5 @@
       <origin xyz="0.125 0.0 0.0255" rpy="0.0 0.0 ${pi}" />
       <axis xyz="0 0 -1" />
-      <limit effort="  2.0" lower="-0.8" upper="-2.9" velocity="10.0" />
+      <limit effort="  2.0" lower="-3.14" upper="3.14" velocity="10.0" />
       <dynamics damping="0.1" friction="0.1" />
     </joint>
