Commit message: Working controller with new mujoco model
Signed-off-by: Jakub Delicat <delicat.kuba@gmail.com>

File: four_bar_bot_description/urdf/four_bar_bot_mujoco.urdf.xacro (robot description, xacro)
@@ -1,3 +1,59 @@
 <?xml version="1.0"?>
+<!-- <mujoco_inputs>
+  <raw_inputs>
+    <equality>
+      <connect anchor="0 0 0" body1="front_left_foot_link" body2="front_left_chain_close_a_link"
+        name="equality_sconstraint_front_left" solref="0.001 2" />
+      <connect anchor="0 0 0" body1="front_right_foot_link" body2="front_right_chain_close_a_link"
+        name="equality_sconstraint_front_right" solref="0.001 2" />
+      <connect anchor="0 0 0" body1="rear_left_foot_link" body2="rear_left_chain_close_a_link"
+        name="equality_sconstraint_rear_left" solref="0.001 2" />
+      <connect anchor="0 0 0" body1="rear_right_foot_link" body2="rear_right_chain_close_a_link"
+        name="equality_sconstraint_rear_right" solref="0.001 2" />
+    </equality>
+    <contact>
+      <exclude body1="front_right_second_link" body2="front_right_third_link" />
+      <exclude body1="front_right_second_link" body2="front_right_fourth_link" />
+      <exclude body1="front_right_second_link" body2="front_right_fifth_link" />
+      <exclude body1="front_right_second_link" body2="front_right_sixth_link" />
+      <exclude body1="front_right_third_link" body2="front_right_fourth_link" />
+      <exclude body1="front_right_third_link" body2="front_right_fifth_link" />
+      <exclude body1="front_right_third_link" body2="front_right_sixth_link" />
+      <exclude body1="front_right_fourth_link" body2="front_right_fifth_link" />
+      <exclude body1="front_right_fourth_link" body2="front_right_sixth_link" />
+      <exclude body1="front_right_fifth_link" body2="front_right_sixth_link" />
+      <exclude body1="front_left_second_link" body2="front_left_third_link" />
+      <exclude body1="front_left_second_link" body2="front_left_fourth_link" />
+      <exclude body1="front_left_second_link" body2="front_left_fifth_link" />
+      <exclude body1="front_left_second_link" body2="front_left_sixth_link" />
+      <exclude body1="front_left_third_link" body2="front_left_fourth_link" />
+      <exclude body1="front_left_third_link" body2="front_left_fifth_link" />
+      <exclude body1="front_left_third_link" body2="front_left_sixth_link" />
+      <exclude body1="front_left_fourth_link" body2="front_left_fifth_link" />
+      <exclude body1="front_left_fourth_link" body2="front_left_sixth_link" />
+      <exclude body1="front_left_fifth_link" body2="front_left_sixth_link" />
+      <exclude body1="rear_right_second_link" body2="rear_right_third_link" />
+      <exclude body1="rear_right_second_link" body2="rear_right_fourth_link" />
+      <exclude body1="rear_right_second_link" body2="rear_right_fifth_link" />
+      <exclude body1="rear_right_second_link" body2="rear_right_sixth_link" />
+      <exclude body1="rear_right_third_link" body2="rear_right_fourth_link" />
+      <exclude body1="rear_right_third_link" body2="rear_right_fifth_link" />
+      <exclude body1="rear_right_third_link" body2="rear_right_sixth_link" />
+      <exclude body1="rear_right_fourth_link" body2="rear_right_fifth_link" />
+      <exclude body1="rear_right_fourth_link" body2="rear_right_sixth_link" />
+      <exclude body1="rear_right_fifth_link" body2="rear_right_sixth_link" />
+      <exclude body1="rear_left_second_link" body2="rear_left_third_link" />
+      <exclude body1="rear_left_second_link" body2="rear_left_fourth_link" />
+      <exclude body1="rear_left_second_link" body2="rear_left_fifth_link" />
+      <exclude body1="rear_left_second_link" body2="rear_left_sixth_link" />
+      <exclude body1="rear_left_third_link" body2="rear_left_fourth_link" />
+      <exclude body1="rear_left_third_link" body2="rear_left_fifth_link" />
+      <exclude body1="rear_left_third_link" body2="rear_left_sixth_link" />
+      <exclude body1="rear_left_fourth_link" body2="rear_left_fifth_link" />
+      <exclude body1="rear_left_fourth_link" body2="rear_left_sixth_link" />
+      <exclude body1="rear_left_fifth_link" body2="rear_left_sixth_link" />
+    </contact>
+  </raw_inputs>
+</mujoco_inputs> -->
 <robot name="quadruped" xmlns:xacro="http://www.ros.org/wiki/xacro">
   <xacro:include filename="$(find four_bar_bot_description)/urdf/inertia.urdf.xacro" />
@@ -6,5 +62,5 @@
   <xacro:arg name="use_hardware" default="True" />
   <xacro:arg name="use_sim" default="False" />
-  <mujoco>
+  <!-- <mujoco>
     <compiler
       balanceinertia="true"
@@ -12,5 +68,5 @@
       discardfixed="false"
       fusestatic="false"/>
-  </mujoco>
+  </mujoco> -->
   <material name="grey">
     <color rgba="0.5 0.5 0.5 1" />

File: four_bar_bot_description/urdf/leg.urdf.xacro (robot description, xacro)
@@ -5,6 +5,4 @@
   <xacro:macro name="leg"
     params="prefix xyz rpy first_x:=0.1 first_joint_offset third_joint_gear_correction_dir ">
-    <xacro:property name="zero_angle_offset" value="0.17692153346630435" />
-    <!-- Define the thigh -->
     <link name="${prefix}_leg_base_link" />
     <!-- Define the joints -->
@@ -37,8 +35,4 @@
       name="${prefix}_third_link" />
     <xacro:property name="gear_ratio" value="0.0" />
-    <!-- <xacro:property name="second_joint_gear_correction" value="${third_joint_gear_correction_dir*0.2793}" />
-    <xacro:property name="third_joint_gear_correction" value="${-1.117+pi}" /> -->
-    <xacro:property name="second_joint_gear_correction" value="0" />
-    <xacro:property name="third_joint_gear_correction" value="${1.198}" />
     <joint name="${prefix}_second_joint"
       type="revolute">
@@ -48,9 +42,15 @@
         rpy="0.0 0.0 ${pi} " />
       <axis xyz="0 0 1" />
-      <limit effort="100.0" lower="1.57" upper="4.71" velocity="10.0" />
+      <limit effort="100.0" lower="-5.8" upper="5.8" velocity="10.0" />
       <dynamics damping="0.1" friction="0.1" />
     </joint>
     <xacro:fourth_link
       name="${prefix}_fourth_link" />
+    <!-- <xacro:property name="second_joint_gear_correction" value="${third_joint_gear_correction_dir*0.2793}" />
+    <xacro:property name="third_joint_gear_correction" value="${-1.117+pi}" /> -->
+    <!-- <xacro:property name="fr_sign" value="${1 if 'front' in prefix else -1}" />
+    <xacro:property name="lr_sign" value="${1 if 'left' in prefix else -1}" />
+    <xacro:property name="third_joint_gear_correction" value="${third_joint_gear_correction_dir*0.7  if third_joint_gear_correction_dir > 0 else third_joint_gear_correction_dir*0.7 -1.198*2.0}" /> -->
+    <xacro:property name="third_joint_gear_correction" value="${pi}" />
     <joint name="${prefix}_third_joint"
       type="revolute">
@@ -58,7 +58,7 @@
       <child link="${prefix}_fourth_link" />
       <origin xyz="0.0 0.0 0.0555"
-        rpy="0.0 0.0 ${third_joint_gear_correction_dir*third_joint_gear_correction}" />
-      <axis xyz="0 0 ${third_joint_gear_correction_dir}" />
-      <limit effort="100.0" lower="0.425" upper="5.8" velocity="10.0" />
+        rpy="0.0 0.0 ${third_joint_gear_correction}" />
+      <axis xyz="0 0 1" />
+      <limit effort="100.0" lower="-5.8" upper="5.8" velocity="10.0" />
       <dynamics damping="0.1" friction="0.1" />
     </joint>
@@ -193,4 +193,18 @@
       <xacro:box_inertia m="0.05" w="0.25" h="0.04" d="0.0175" xyz="0.105 0  0.0" />
     </link>
+    <!-- Punkt zamknięcia pętli od strony aktywnej gałęzi (fifth_link) -->
+    <link name="${prefix}_chain_close_a_link" />
+    <joint name="${prefix}_chain_close_a_joint" type="fixed">
+      <parent link="${prefix}_fifth_link" />
+      <child link="${prefix}_chain_close_a_link" />
+      <origin xyz="0.21 0 -0.0115" rpy="0 0 0" />
+    </joint>
+    <!-- Punkt zamknięcia pętli od strony pasywnej gałęzi (sixth_link) -->
+    <link name="${prefix}_foot_link" />
+    <joint name="${prefix}_foot_joint" type="fixed">
+      <parent link="${prefix}_sixth_link" />
+      <child link="${prefix}_foot_link" />
+      <origin xyz="0.21 0 0.0115" rpy="0 0 0" />
+    </joint>
   </xacro:macro>
 </robot>

File: four_bar_bot_description/urdf/ros2_control.urdf.xacro (robot description, xacro)
@@ -5,8 +5,11 @@
               q_kp=10.0   q_ki=0.5    q_kd=0.0    q_windup=1.0
               dq_kp=2.0   dq_ki=0.5   dq_kd=0.0   dq_windup=0.1
-              ddq_kp=1.0  ddq_kd=0.15">
+              ddq_kp=1.0  ddq_kd=0.15 init_pos=0.0">
         <joint name="${name}">
             <xacro:if value="${use_hardware}">
-                <command_interface name="effort" />
+                    <command_interface name="effort">
+                        <param name="min">-20.0</param>
+                        <param name="max">20.0</param>
+                    </command_interface>
             </xacro:if>
             <xacro:unless value="${use_hardware}">
@@ -14,5 +17,5 @@
             </xacro:unless>
             <state_interface name="position">
-                <param name="initial_value">0.0</param>
+                <param name="initial_value">${init_pos}</param>
             </state_interface>
             <state_interface name="velocity">
@@ -63,19 +66,28 @@
         <ros2_control name="MD80HardwareInterface" type="system">
             <hardware>
+                <!-- mock params -->
+                <!-- <plugin>mock_components/GenericSystem</plugin>
+                <param name="calculate_dynamics">false</param>
+                <param name="custom_interface_with_following_offset"></param>
+                <param name="disable_commands">false</param>
+                <param name="mock_gpio_commands">false</param>
+                <param name="mock_sensor_commands">true</param>
+                <param name="position_state_following_offset">0.0</param> -->
                 <plugin>mujoco_ros2_control/MujocoSystemInterface</plugin>
                 <param name="mujoco_model">$(find four_bar_bot_mujoco)/config/mujoco_description_formatted.xml</param>
                 <param name="sim_speed_factor">1.0</param>
+                <param name="headless">false</param>
             </hardware>
             <xacro:property name="kp1" value="25" />
             <xacro:property name="kd1" value="5.0" />
-            <xacro:property name="max_torque1" value="2.0" />
+            <xacro:property name="max_torque1" value="20.0" />
             <!-- <xacro:property name="kp2" value="50" /> -->
             <xacro:property name="kp2" value="7.5" />
             <xacro:property name="kd2" value="1.0" />
-            <xacro:property name="max_torque2" value="1.0" />
+            <xacro:property name="max_torque2" value="10.0" />
             <!-- <xacro:property name="kp3" value="50" /> -->
             <xacro:property name="kp3" value="7.5" />
             <xacro:property name="kd3" value="1.0" />
-            <xacro:property name="max_torque3" value="1.0" />
+            <xacro:property name="max_torque3" value="10.0" />
             <xacro:ros2_control_joint_can name="front_left_first_joint" can_id="10" use_hardware="${use_hardware}" ddq_kp="${kp1}"
                 ddq_kd="${kd1}" max_torque="${max_torque1}" />
@@ -83,5 +95,5 @@
                 ddq_kd="${kd2}" max_torque="${max_torque2}" />
             <xacro:ros2_control_joint_can name="front_left_third_joint" can_id="12" use_hardware="${use_hardware}" ddq_kp="${kp3}"
-                ddq_kd="${kd3}" max_torque="${max_torque3}" />
+                ddq_kd="${kd3}" max_torque="${max_torque3}" init_pos="${pi/2}" />
             <xacro:ros2_control_joint_can name="front_right_first_joint" can_id="20" use_hardware="${use_hardware}"  ddq_kp="${kp1}"
                 ddq_kd="${kd1}" max_torque="${max_torque1}" />
@@ -90,5 +102,5 @@
                 ddq_kd="${kd2}" max_torque="${max_torque2}" />
             <xacro:ros2_control_joint_can name="front_right_third_joint" can_id="22" use_hardware="${use_hardware}" ddq_kp="${kp3}"
-                ddq_kd="${kd3}" max_torque="${max_torque3}" />
+                ddq_kd="${kd3}" max_torque="${max_torque3}" init_pos="${pi/2}" />
             <xacro:ros2_control_joint_can name="rear_right_first_joint" can_id="30" use_hardware="${use_hardware}" ddq_kp="${kp1}"
                 ddq_kd="${kd1}" max_torque="${max_torque1}" />
@@ -96,5 +108,5 @@
                 ddq_kd="${kd2}" max_torque="${max_torque2}" />
             <xacro:ros2_control_joint_can name="rear_right_third_joint" can_id="32" use_hardware="${use_hardware}" ddq_kp="${kp3}"
-                ddq_kd="${kd3}" max_torque="${max_torque3}" />
+                ddq_kd="${kd3}" max_torque="${max_torque3}" init_pos="${pi/2}" />
             <xacro:ros2_control_joint_can name="rear_left_first_joint" can_id="40" use_hardware="${use_hardware}" ddq_kp="${kp1}"
                 ddq_kd="${kd1}" max_torque="${max_torque1}" />
@@ -102,5 +114,5 @@
                 ddq_kd="${kd2}" max_torque="${max_torque2}" />
             <xacro:ros2_control_joint_can name="rear_left_third_joint" can_id="42" use_hardware="${use_hardware}" ddq_kp="${kp3}"
-                ddq_kd="${kd3}" max_torque="${max_torque3}" />
+                ddq_kd="${kd3}" max_torque="${max_torque3}" init_pos="${pi/2}" />
         </ros2_control>
     </xacro:macro>
